File: Kicad/motors/motors.kicad_pcb (KiCad board)
At the start: 2 copper layers, 80 x 140 mm, 137 parts, among them IC100 BQ2057W, IC201 L298P, IC202 SN74LVC1G19, IC203 SN74LVC1G19, IC204 L298P, IC205 SN74LVC1G19, IC206 SN74LVC1G19, IC207 LM3480-50, IC301 SN74LVC2G17, IC302 SN74LVC2G17, IC303 OPB610, IC304 OPB610, IC305 OPB610, IC306 OPB610, IC307 LM3480-33, K100 Charger, K201 MOTOR 1, K202 MOTOR 2, K203 MOTOR 4, K204 MOTOR 3, K301 Front, K302 Rear, Q100 STN790A, Q301 BC846B, Q302 BC846B, Q303 BC846B, Q304 BC846B, T101 DMP2305U, T102 DMP2305U

Commit message: Update Motors
Parts:
- IC303, IC304, IC305, IC306: value OPB610 -> TTE-OPB610
Changed lines of the file:
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@@
   (net 65 "ENCODER_M1")
   (net 66 "/Driver/M2+")
-  (net 67 "Net-(IC305-Pad2)")
-  (net 68 "Net-(IC306-Pad2)")
+  (net 67 "Net-(Q301-Pad3)")
+  (net 68 "Net-(Q302-Pad3)")
   (net 69 "unconnected-(IC201-Pad3)")
   (net 70 "unconnected-(IC201-Pad18)")
@@
       (net 49 "Net-(Q301-Pad2)") (pinfunction "E") (pintype "passive"))
     (pad "3" smd roundrect (at 1.2 0 90) (size 1.2 0.8) (layers "F.Cu" "F.Paste" "F.Mask") (roundrect_rratio 0.25)
-      (net 67 "Net-(IC305-Pad2)") (pinfunction "C") (pintype "passive"))
+      (net 67 "Net-(Q301-Pad3)") (pinfunction "C") (pintype "passive"))
     (model "${KICAD6_USER_3DMODEL_DIR}/SMD/SOT-23.wrl"
       (offset (xyz 0 0 0))
@@
       (net 52 "Net-(Q302-Pad2)") (pinfunction "E") (pintype "passive"))
     (pad "3" smd roundrect (at 1.2 0 270) (size 1.2 0.8) (layers "F.Cu" "F.Paste" "F.Mask") (roundrect_rratio 0.25)
-      (net 68 "Net-(IC306-Pad2)") (pinfunction "C") (pintype "passive"))
+      (net 68 "Net-(Q302-Pad3)") (pinfunction "C") (pintype "passive"))
     (model "${KICAD6_USER_3DMODEL_DIR}/SMD/SOT-23.wrl"
       (offset (xyz 0 0 0))
@@
   (footprint "tronixio:zzzOPB-610" (layer "B.Cu")
     (at 110.5 42.25)
-    (property "MOUSER" "828-OPB610")
+    (property "Mouser" "828-OPB610")
+    (property "Name" "OPB610")
     (property "Sheetfile" "encoder.kicad_sch")
     (property "Sheetname" "Encoder")
@@
       (effects (font (size 1 1) (thickness 0.15)) (justify mirror))
     )
-    (fp_text value "OPB610" (at 0 -5.08) (layer "B.Fab")
+    (fp_text value "TTE-OPB610" (at 0 -5.08) (layer "B.Fab")
       (effects (font (size 1 1) (thickness 0.15)) (justify mirror))
     )
@@
     (fp_line (start -1.2 -0.4) (end -1.2 -3) (layer "B.Fab") (width 0.1))
     (pad "1" thru_hole circle (at -3.5 1.27) (size 1.6 1.6) (drill 0.7) (layers *.Cu *.Mask)
-      (net 50 "Net-(IC303-Pad2)") (pinfunction "LEDA") (pintype "passive"))
+      (net 50 "Net-(IC303-Pad2)") (pinfunction "ANODE") (pintype "passive"))
     (pad "2" thru_hole circle (at -3.5 -1.27) (size 1.6 1.6) (drill 0.7) (layers *.Cu *.Mask)
-      (net 67 "Net-(IC305-Pad2)") (pinfunction "LEDC") (pintype "passive"))
+      (net 67 "Net-(Q301-Pad3)") (pinfunction "CATHODE") (pintype "passive"))
     (pad "3" thru_hole circle (at 3.5 -1.27) (size 1.6 1.6) (drill 0.7) (layers *.Cu *.Mask)
-      (net 5 "Net-(IC301-Pad3)") (pinfunction "TRC") (pintype "passive"))
+      (net 5 "Net-(IC301-Pad3)") (pinfunction "COLLECTOR") (pintype "passive"))
     (pad "4" thru_hole circle (at 3.5 1.27) (size 1.6 1.6) (drill 0.7) (layers *.Cu *.Mask)
-      (net 1 "GND") (pinfunction "TRE") (pintype "passive"))
+      (net 1 "GND") (pinfunction "EMITTER") (pintype "passive"))
     (model "${KICAD6_USER_3DMODEL_DIR}/Opto/TTE-OBP610.step"
       (offset (xyz 0 0 0))
@@
   (footprint "tronixio:zzzOPB-610" (layer "B.Cu")
     (at 110.5 157.75 180)
-    (property "MOUSER" "828-OPB610")
+    (property "Mouser" "828-OPB610")
+    (property "Name" "OPB610")
     (property "Sheetfile" "encoder.kicad_sch")
     (property "Sheetname" "Encoder")
@@
       (effects (font (size 1 1) (thickness 0.15)) (justify mirror))
     )
-    (fp_text value "OPB610" (at 0 -5.08) (layer "B.Fab")
+    (fp_text value "TTE-OPB610" (at 0 -5.08) (layer "B.Fab")
       (effects (font (size 1 1) (thickness 0.15)) (justify mirror))
     )
@@
     (fp_line (start 1.7 -0.4) (end 1.7 0.4) (layer "B.Fab") (width 0.1))
     (pad "1" thru_hole circle (at -3.5 1.27 180) (size 1.6 1.6) (drill 0.7) (layers *.Cu *.Mask)
-      (net 2 "VIN") (pinfunction "LEDA") (pintype "passive"))
+      (net 2 "VIN") (pinfunction "ANODE") (pintype "passive"))
     (pad "2" thru_hole circle (at -3.5 -1.27 180) (size 1.6 1.6) (drill 0.7) (layers *.Cu *.Mask)
-      (net 53 "Net-(IC304-Pad2)") (pinfunction "LEDC") (pintype "passive"))
+      (net 53 "Net-(IC304-Pad2)") (pinfunction "CATHODE") (pintype "passive"))
     (pad "3" thru_hole circle (at 3.5 -1.27 180) (size 1.6 1.6) (drill 0.7) (layers *.Cu *.Mask)
-      (net 37 "Net-(IC302-Pad1)") (pinfunction "TRC") (pintype "passive"))
+      (net 37 "Net-(IC302-Pad1)") (pinfunction "COLLECTOR") (pintype "passive"))
     (pad "4" thru_hole circle (at 3.5 1.27 180) (size 1.6 1.6) (drill 0.7) (layers *.Cu *.Mask)
-      (net 1 "GND") (pinfunction "TRE") (pintype "passive"))
+      (net 1 "GND") (pinfunction "EMITTER") (pintype "passive"))
     (model "${KICAD6_USER_3DMODEL_DIR}/Opto/TTE-OBP610.step"
       (offset (xyz 0 0 0))
@@
   (footprint "tronixio:zzzOPB-610" (layer "B.Cu")
     (at 67.5 157.75 180)
-    (property "MOUSER" "828-OPB610")
+    (property "Mouser" "828-OPB610")
+    (property "Name" "OPB610")
     (property "Sheetfile" "encoder.kicad_sch")
     (property "Sheetname" "Encoder")
@@
       (effects (font (size 1 1) (thickness 0.15)) (justify mirror))
     )
-    (fp_text value "OPB610" (at 0 -5.08) (layer "B.Fab")
+    (fp_text value "TTE-OPB610" (at 0 -5.08) (layer "B.Fab")
       (effects (font (size 1 1) (thickness 0.15)) (justify mirror))
     )
@@
     (fp_line (start -1.7 0.4) (end -1.7 -0.4) (layer "B.Fab") (width 0.1))
     (pad "1" thru_hole circle (at -3.5 1.27 180) (size 1.6 1.6) (drill 0.7) (layers *.Cu *.Mask)
-      (net 53 "Net-(IC304-Pad2)") (pinfunction "LEDA") (pintype "passive"))
+      (net 53 "Net-(IC304-Pad2)") (pinfunction "ANODE") (pintype "passive"))
     (pad "2" thru_hole circle (at -3.5 -1.27 180) (size 1.6 1.6) (drill 0.7) (layers *.Cu *.Mask)
-      (net 68 "Net-(IC306-Pad2)") (pinfunction "LEDC") (pintype "passive"))
+      (net 68 "Net-(Q302-Pad3)") (pinfunction "CATHODE") (pintype "passive"))
     (pad "3" thru_hole circle (at 3.5 -1.27 180) (size 1.6 1.6) (drill 0.7) (layers *.Cu *.Mask)
-      (net 38 "Net-(IC302-Pad3)") (pinfunction "TRC") (pintype "passive"))
+      (net 38 "Net-(IC302-Pad3)") (pinfunction "COLLECTOR") (pintype "passive"))
     (pad "4" thru_hole circle (at 3.5 1.27 180) (size 1.6 1.6) (drill 0.7) (layers *.Cu *.Mask)
-      (net 1 "GND") (pinfunction "TRE") (pintype "passive"))
+      (net 1 "GND") (pinfunction "EMITTER") (pintype "passive"))
     (model "${KICAD6_USER_3DMODEL_DIR}/Opto/TTE-OBP610.step"
       (offset (xyz 0 0 0))
@@
   (footprint "tronixio:zzzOPB-610" (layer "B.Cu")
     (at 67.5 42.25)
-    (property "MOUSER" "828-OPB610")
+    (property "Mouser" "828-OPB610")
+    (property "Name" "OPB610")
     (property "Sheetfile" "encoder.kicad_sch")
     (property "Sheetname" "Encoder")
@@
       (effects (font (size 1 1) (thickness 0.15)) (justify mirror))
     )
-    (fp_text value "OPB610" (at 0 -5.08) (layer "B.Fab")
+    (fp_text value "TTE-OPB610" (at 0 -5.08) (layer "B.Fab")
       (effects (font (size 1 1) (thickness 0.15)) (justify mirror))
     )
@@
     (fp_line (start 1.7 -0.4) (end 1.7 0.4) (layer "B.Fab") (width 0.1))
     (pad "1" thru_hole circle (at -3.5 1.27) (size 1.6 1.6) (drill 0.7) (layers *.Cu *.Mask)
-      (net 2 "VIN") (pinfunction "LEDA") (pintype "passive"))
+      (net 2 "VIN") (pinfunction "ANODE") (pintype "passive"))
     (pad "2" thru_hole circle (at -3.5 -1.27) (size 1.6 1.6) (drill 0.7) (layers *.Cu *.Mask)
-      (net 50 "Net-(IC303-Pad2)") (pinfunction "LEDC") (pintype "passive"))
+      (net 50 "Net-(IC303-Pad2)") (pinfunction "CATHODE") (pintype "passive"))
     (pad "3" thru_hole circle (at 3.5 -1.27) (size 1.6 1.6) (drill 0.7) (layers *.Cu *.Mask)
-      (net 35 "Net-(IC301-Pad1)") (pinfunction "TRC") (pintype "passive"))
+      (net 35 "Net-(IC301-Pad1)") (pinfunction "COLLECTOR") (pintype "passive"))
     (pad "4" thru_hole circle (at 3.5 1.27) (size 1.6 1.6) (drill 0.7) (layers *.Cu *.Mask)
-      (net 1 "GND") (pinfunction "TRE") (pintype "passive"))
+      (net 1 "GND") (pinfunction "EMITTER") (pintype "passive"))
     (model "${KICAD6_USER_3DMODEL_DIR}/Opto/TTE-OBP610.step"
       (offset (xyz 0 0 0))

Commit message: Update Motor
Parts:
- removed Q303, Q304: BC846B, tronixio:SOT-23-3
- removed T101, T102: DMP2305U, tronixio:SOT-23-3
- added Q101: DMP2305U, tronixio:SOT-23-3, B.Cu at (60.0, 84.0)
- added Q102: STN790A, tronixio:SOT-223-3, B.Cu at (89.0, 95.0)
- Q100: value STN790A -> DMP2305U; footprint tronixio:SOT-223-3 -> tronixio:SOT-23-3
- Q301, Q302: value BC846B -> NEXPERIA-BC846BS; footprint tronixio:SOT-23-3 -> tronixio:zzzSOT-70-6
- R208: footprint tronixio:RESISTOR-1206 -> tronixio:RESISTOR-1210
- moved Q100 37.7 mm to (52.9, 84.0), turned to -90 degrees
- moved Q301 0.50 mm to (117.5, 42.2), turned to 0 degrees
- moved Q302 0.50 mm to (60.5, 157.8), turned to 180 degrees
- turned R307 to -90 degrees
Connections:
- IC305 pad 2: Net-(Q301-Pad3) -> Net-(IC305-Pad2)
- IC306 pad 2: Net-(Q302-Pad3) -> Net-(IC306-Pad2)
- Q100 pad 1: Net-(Q100-Pad1) -> GND
- Q100 pad 2: VBAT -> Net-(Q100-Pad2)
- Q100 pad 3: Net-(IC100-Pad1) -> VBAT
- Q301 pad 3: Net-(Q301-Pad3) -> Net-(Q301-Pad2)
- Q302 pad 3: Net-(Q302-Pad3) -> Net-(Q302-Pad2)
- R102 pad 1: Net-(Q100-Pad1) -> Net-(Q102-Pad1)
- R104 pad 2: Net-(R104-Pad2) -> Net-(Q100-Pad2)
- R305 pad 2: Net-(Q301-Pad1) -> Net-(Q301-Pad2)
- R306 pad 2: Net-(Q302-Pad1) -> Net-(Q302-Pad2)
- R307 pad 1: Net-(Q301-Pad2) -> Net-(Q301-Pad1)
- R308 pad 1: Net-(Q302-Pad2) -> Net-(Q302-Pad1)
Routing:
- net Net-(Q302-Pad1): track 37.9 -> 5.57 mm
- net Net-(Q301-Pad1): track 37.6 -> 5.57 mm
- net Net-(Q301-Pad2): track 5.35 -> 29.8 mm
- net Net-(Q302-Pad2): track 5.35 -> 29.4 mm
- net GND: track 187.3 -> 171.0 mm, vias 58 -> 59
- net Net-(IC305-Pad2): track 0.00 -> 13.5 mm
- net Net-(IC306-Pad2): track 0.00 -> 13.3 mm
- net Net-(Q301-Pad3): track 12.1 -> 0.00 mm
- net Net-(Q302-Pad3): track 11.9 -> 0.00 mm
- net Net-(R104-Pad2): track 7.23 -> 0.00 mm
- net Net-(Q100-Pad2): track 0.00 -> 7.23 mm
- net Net-(Q102-Pad1): track 0.00 -> 5.65 mm
- net Net-(Q100-Pad1): track 5.65 -> 0.00 mm
- net +5V: track 195.0 -> 196.0 mm
