File: Kicad/motors/motors.kicad_pcb (KiCad board)
At the start: 2 copper layers, 80 x 140 mm, 135 parts, among them IC100 BQ2057W, IC201 L298P, IC202 SN74LVC1G19, IC203 SN74LVC1G19, IC204 L298P, IC205 SN74LVC1G19, IC206 SN74LVC1G19, IC207 LM3480-50, IC301 SN74LVC2G17, IC302 SN74LVC2G17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

Commit message: Update
Parts:
- added TP104: KEYSTONE-2000-3, tronixio:KEYSTONE-2000-3, F.Cu at (52.5, 158.5)
- added TP105: KEYSTONE-2000-3, tronixio:KEYSTONE-2000-3, F.Cu at (125.5, 41.5)
- added kibuzzard-62897416: G***, kibuzzard-62897416, F.Cu at (77.6, 36.0)
- added kibuzzard-628974BE: G***, kibuzzard-628974BE, F.Cu at (100.5, 36.0)
- added kibuzzard-62897505: G***, kibuzzard-62897505, F.Cu at (77.6, 164.0)
- added kibuzzard-6289753B: G***, kibuzzard-6289753B, F.Cu at (100.5, 164.0)
- added kibuzzard-6289769F: G***, kibuzzard-6289769F, F.Cu at (125.5, 44.0)
- added kibuzzard-6289769F: G***, kibuzzard-6289769F, F.Cu at (52.5, 156.0)
- added kibuzzard-628977DB: G***, kibuzzard-628977DB, F.Cu at (125.5, 67.5)
- added kibuzzard-628977F0: G***, kibuzzard-628977F0, F.Cu at (52.5, 67.5)
- added kibuzzard-62897802: G***, kibuzzard-62897802, F.Cu at (52.5, 44.0)
- added kibuzzard-6289784D: G***, kibuzzard-6289784D, F.Cu at (125.5, 156.0)
- added kibuzzard-6289786A: G***, kibuzzard-6289786A, F.Cu at (52.5, 132.5)
- added kibuzzard-62897881: G***, kibuzzard-62897881, F.Cu at (125.5, 132.5)
- D100, D201, D202, D203, D204, D205, D206, D207, D208, D209, D210, D211, D212, D213, D214, D215, D216: value PMEG3030 -> NEXPERIA-PMEG3030
- LED100: value Charging -> LED-1206-RED
- LED101: value Power -> LED-1206-RED
- LED201, LED202, LED203, LED204, LED205, LED206, LED207, LED208: value Red -> LED-1206-RED
- LED209: value +5V -> LED-1206-RED
- LED301: value +3V3 -> LED-1206-RED
- Q100, Q101: value DMP2305U -> DIODESINC-DMP2305U-SOT-23
- Q102: value STN790A -> ST-STN790A
- turned TP102 to 0 degrees
Routing:
- net GND: track 171.0 -> 173.2 mm
Other:
- board text removed: "GND"
- board text removed: "VBAT"
- board text removed: "VIN"

Commit message: Update
Parts:
- removed IC100: BQ2057W, tronixio:SOIC-08
- removed IC201, IC204: L298P, tronixio:zzzSOPOWER-20
- removed IC202, IC203, IC205, IC206: SN74LVC1G19, tronixio:SOT-23-6
- removed IC207: LM3480-50, tronixio:SOT-23-3
- removed IC301, IC302: SN74LVC2G17, tronixio:SOT-23-6
- removed IC303, IC304, IC305, IC306: TTE-OPB610, tronixio:zzzOPB-610
- removed IC307: LM3480-33, tronixio:SOT-23-3
- added IR301: OPB610, tronixioZZZ:OPB-610, B.Cu at (67.5, 42.2)
- added IR302: OPB610, tronixioZZZ:OPB-610, B.Cu at (110.5, 157.8)
- added IR303: OPB610, tronixioZZZ:OPB-610, B.Cu at (110.5, 42.2)
- added IR304: OPB610, tronixioZZZ:OPB-610, B.Cu at (67.5, 157.8)
- added U100: BQ2057W, tronixio:SOIC-08, B.Cu at (89.0, 103.5)
- added U201: L298P, tronixioZZZ:SOPOWER-20, F.Cu at (89.0, 59.0)
- added U202: SN74LVC1G19, tronixio:SOT-23-6, F.Cu at (75.0, 64.5)
- added U203: SN74LVC1G19, tronixio:SOT-23-6, F.Cu at (103.0, 60.6)
- added U204: L298P, tronixioZZZ:SOPOWER-20, F.Cu at (89.0, 141.0)
- added U205: SN74LVC1G19, tronixio:SOT-23-6, F.Cu at (103.0, 135.5)
- added U206: SN74LVC1G19, tronixio:SOT-23-6, F.Cu at (75.0, 139.4)
- added U207: LM3480-50, tronixio:SOT-23-3, F.Cu at (89.0, 74.5)
- added U301: SN74LVC2G17, tronixio:SOT-23-6, F.Cu at (89.0, 42.2)
- added U302: SN74LVC2G17, tronixio:SOT-23-6, F.Cu at (89.0, 157.8)
- added U303: LM3480-33, tronixio:SOT-23-3, F.Cu at (89.0, 125.5)
- BT100: value 2x18650 -> 18650
- C100, C101, C201, C202, C205, C206, C209, C210, C211, C212, C301, C302, C303, C304, C305, C306: footprint tronixio:CAPACITOR-1206 -> tronixio:CAPACITOR-SMD-1206
- C203, C204, C207, C208: value UVZ-470U-35V -> 470µ/35V; footprint tronixio:zzzCAPACITOR-ELECTROLYTIC-RADIAL-100-160-050 -> tronixioZZZ:CAPACITOR-ELECTROLYTIC-RADIAL-100-160-050
- D100, D201, D202, D203, D204, D205, D206, D207, D208, D209, D210, D211, D212, D213, D214, D215, D216: value NEXPERIA-PMEG3030 -> PMEG3030
- H101, H102, H103, H104, H105, H106, H107, H108, H109, H110, H111, H112, H113, H114, H115, H116: value MOUNTING-HOLE-MASK-3MM -> MOUNTING-HOLE-3MM-MASK; footprint tronixio:M3-MASK -> tronixio:MOUNTING-HOLE-3MM-MASK
- H117, H118, H119, H120: value MOUNTING-HOLE-MASK-3MM -> MOUNTING-HOLE-3.5MM; footprint tronixio:M3.5 -> tronixio:MOUNTING-HOLE-3.5MM
- K100: value Charger -> CHARGER; footprint tronixio:zzzCUI-PJ-002AH-SMT-TR -> tronixioZZZ:CUI-PJ-002AH-SMT-TR
- K301: value Front -> FRONT; footprint tronixio:zzHARWIN-M20-782104x -> tronixio:HARWIN-M20-782104x
- K302: value Rear -> REAR; footprint tronixio:zzHARWIN-M20-782104x -> tronixio:HARWIN-M20-782104x
- LED100: value LED-1206-RED -> CHARGE; footprint tronixio:LED-1206 -> tronixio:LED-SMD-1206
- LED101: value LED-1206-RED -> POWER; footprint tronixio:LED-1206 -> tronixio:LED-SMD-1206
- LED201, LED202, LED203, LED204, LED205, LED206, LED207, LED208: value LED-1206-RED -> KINGBRIGHT-LED-1206-ORANGE; footprint tronixio:LED-1206 -> tronixio:LED-SMD-1206
- LED209: value LED-1206-RED -> +5V; footprint tronixio:LED-1206 -> tronixio:LED-SMD-1206
- LED301: value LED-1206-RED -> +3V3; footprint tronixio:LED-1206 -> tronixio:LED-SMD-1206
- Q100, Q101: value DIODESINC-DMP2305U-SOT-23 -> DMP2305U
- Q102: value ST-STN790A -> STN790A
- Q301, Q302: value NEXPERIA-BC846BS -> BC846BS; footprint tronixio:zzzSOT-70-6 -> tronixioZZZ:SOT-70-6
- R100, R101, R204, R205, R209, R210: footprint tronixio:RESISTOR-1210 -> tronixio:RESISTOR-SMD-1210
- R102, R103, R104, R105, R106, R107, R201, R202, R203, R206, R207, R211, R301, R302, R303, R304, R305, R306, R307, R308, R309: footprint tronixio:RESISTOR-1206 -> tronixio:RESISTOR-SMD-1206
- R208: footprint tronixio:RESISTOR-1210 -> tronixio:RESISTOR-SMD-1206
- S100: value On/Off -> ON/OFF; footprint tronixio:zzzE-SWITCH-200USPXT1A1M6RE -> tronixioZZZ:E-SWITCH-200USPXT1A1M6RE
- TH100: value 10K -> NTC-10K; footprint tronixio:THERMISTOR -> tronixio:THERMISTOR-SMD
- TP100, TP101, TP102, TP103, TP201, TP301: footprint tronixio:zzzHARWIN-S1751 -> tronixioZZZ:HARWIN-S1751
Routing:
- net Net-(IR302-Pad2): track 0.00 -> 47.3 mm
- net Net-(IR301-Pad2): track 0.00 -> 47.3 mm
- net Net-(IC304-Pad2): track 47.3 -> 0.00 mm
- net Net-(IC303-Pad2): track 47.3 -> 0.00 mm
- net Net-(U204-Pad7): track 0.00 -> 6.70 mm
- net Net-(IC204-Pad7): track 6.70 -> 0.00 mm
- net Net-(U201-Pad7): track 0.00 -> 6.70 mm
- net Net-(IC201-Pad7): track 6.70 -> 0.00 mm
- net Net-(U201-Pad9): track 0.00 -> 6.43 mm
- net Net-(IC201-Pad9): track 6.43 -> 0.00 mm
- net Net-(U204-Pad9): track 0.00 -> 6.43 mm
- net Net-(IC204-Pad9): track 6.43 -> 0.00 mm
- net Net-(U204-Pad13): track 0.00 -> 5.87 mm
- net Net-(IC204-Pad13): track 5.87 -> 0.00 mm
- net Net-(U201-Pad13): track 0.00 -> 5.87 mm
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Other:
- board text added: "GND"
- board text added: "VIN"

Commit message: Update
Parts:
- K100: value CHARGER -> 9V - 1A
- TP104, TP105: footprint tronixio:KEYSTONE-2000-3 -> tronixioZZZ:HARWIN-S1751
Routing:
- net GND: track 173.2 -> 177.2 mm, vias 59 -> 61
Changed lines of the file:
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@@
     )
   )
-  (footprint "tronixio:KEYSTONE-2000-3" (layer "F.Cu")
+  (footprint "tronixioZZZ:HARWIN-S1751" (layer "F.Cu")
     (at 125.5 41.5)
-    (property "Mouser" "534-2000-3")
-    (property "Name" "KEYSTONE-2000-3")
+    (property "Mouser" "855-S1751-46")
+    (property "Name" "HARWIN-S1751")
     (property "Sheetfile" "motors.kicad_sch")
     (property "Sheetname" "")
-    (attr through_hole)
-    (fp_text reference "TP105" (at 0 -2.54) (layer "F.Fab")
+    (zone_connect 2)
+    (attr smd)
+    (fp_text reference "TP105" (at 0 -2.5) (layer "F.Fab")
       (effects (font (size 1 1) (thickness 0.15)))
     )
-    (fp_text value "KEYSTONE-2000-3" (at 0 2.54) (layer "F.Fab")
+    (fp_text value "KEYSTONE-2000-3" (at 0 2.5) (layer "F.Fab")
       (effects (font (size 1 1) (thickness 0.15)))
     )
-    (fp_circle (center 0 0) (end 1 0) (layer "F.SilkS") (width 0.15) (fill none))
-    (fp_circle (center 0 0) (end 1 0) (layer "F.CrtYd") (width 0.05) (fill none))
-    (fp_circle (center 0 0) (end 1 0) (layer "F.Fab") (width 0.1) (fill none))
-    (pad "1" thru_hole circle (at 0 0) (size 1.4 1.4) (drill 0.5) (layers *.Cu *.Mask)
-      (net 1 "GND") (pinfunction "1") (pintype "passive"))
-    (model "${KICAD6_USER_3DMODEL_DIR}/Discret/KEYSTONE-2000-3.step"
-      (offset (xyz 0 0 -2.6))
+    (fp_rect (start -2 1.3) (end 2 -1.3) (layer "F.SilkS") (width 0.15) (fill none))
+    (fp_rect (start -2 1.3) (end 2 -1.3) (layer "F.CrtYd") (width 0.05) (fill none))
+    (fp_rect (start -2 1.3) (end 2 -1.3) (layer "F.Fab") (width 0.1) (fill none))
+    (pad "1" smd roundrect (at 0 0) (size 3.5 2) (layers "F.Cu" "F.Paste" "F.Mask") (roundrect_rratio 0.1)
+      (net 1 "GND") (pinfunction "1") (pintype "passive") (zone_connect 2))
+    (model "${KICAD6_USER_3DMODEL_DIR}/SMD/HARWIN-S1751.step"
+      (offset (xyz 0 0.8 2))
       (scale (xyz 1 1 1))
       (rotate (xyz -90 0 0))
@@
       (solder_mask_margin 1.5) (clearance 1.5))
   )
-  (footprint "tronixio:KEYSTONE-2000-3" (layer "F.Cu")
+  (footprint "tronixioZZZ:HARWIN-S1751" (layer "F.Cu")
     (at 52.5 158.5)
-    (property "Mouser" "534-2000-3")
-    (property "Name" "KEYSTONE-2000-3")
+    (property "Mouser" "855-S1751-46")
+    (property "Name" "HARWIN-S1751")
     (property "Sheetfile" "motors.kicad_sch")
     (property "Sheetname" "")
-    (attr through_hole)
-    (fp_text reference "TP104" (at 0 -2.54) (layer "F.Fab")
+    (zone_connect 2)
+    (attr smd)
+    (fp_text reference "TP104" (at 0 -2.5) (layer "F.Fab")
       (effects (font (size 1 1) (thickness 0.15)))
     )
-    (fp_text value "KEYSTONE-2000-3" (at 0 2.54) (layer "F.Fab")
+    (fp_text value "KEYSTONE-2000-3" (at 0 2.5) (layer "F.Fab")
       (effects (font (size 1 1) (thickness 0.15)))
     )
-    (fp_circle (center 0 0) (end 1 0) (layer "F.SilkS") (width 0.15) (fill none))
-    (fp_circle (center 0 0) (end 1 0) (layer "F.CrtYd") (width 0.05) (fill none))
-    (fp_circle (center 0 0) (end 1 0) (layer "F.Fab") (width 0.1) (fill none))
-    (pad "1" thru_hole circle (at 0 0) (size 1.4 1.4) (drill 0.5) (layers *.Cu *.Mask)
-      (net 1 "GND") (pinfunction "1") (pintype "passive"))
-    (model "${KICAD6_USER_3DMODEL_DIR}/Discret/KEYSTONE-2000-3.step"
-      (offset (xyz 0 0 -2.6))
+    (fp_rect (start -2 1.3) (end 2 -1.3) (layer "F.SilkS") (width 0.15) (fill none))
+    (fp_rect (start -2 1.3) (end 2 -1.3) (layer "F.CrtYd") (width 0.05) (fill none))
+    (fp_rect (start -2 1.3) (end 2 -1.3) (layer "F.Fab") (width 0.1) (fill none))
+    (pad "1" smd roundrect (at 0 0) (size 3.5 2) (layers "F.Cu" "F.Paste" "F.Mask") (roundrect_rratio 0.1)
+      (net 1 "GND") (pinfunction "1") (pintype "passive") (zone_connect 2))
+    (model "${KICAD6_USER_3DMODEL_DIR}/SMD/HARWIN-S1751.step"
+      (offset (xyz 0 0.8 2))
       (scale (xyz 1 1 1))
       (rotate (xyz -90 0 0))
@@
       (effects (font (size 1 1) (thickness 0.15)) (justify mirror))
     )
-    (fp_text value "CHARGER" (at 0 -1.27 90) (layer "B.Fab")
+    (fp_text value "9V - 1A" (at 0 -1.27 90) (layer "B.Fab")
       (effects (font (size 1 1) (thickness 0.15)) (justify mirror))
     )
@@
   (segment (start 104.5 65.5) (end 106.75 65.5) (width 0.5) (layer "F.Cu") (net 1))
   (segment (start 119 44) (end 118.45 44) (width 0.5) (layer "F.Cu") (net 1))
+  (segment (start 125.5 41.5) (end 125.5 39.5) (width 0.8) (layer "F.Cu") (net 1))
   (segment (start 72.5 62) (end 72.5 64.5) (width 0.5) (layer "F.Cu") (net 1))
   (segment (start 85.5 76) (end 87 76) (width 0.5) (layer "F.Cu") (net 1))
@@
   (segment locked (start 89 75.7) (end 90.7 75.7) (width 0.5) (layer "F.Cu") (net 1))
   (segment (start 101.5 150.5) (end 104.5 147.5) (width 0.8) (layer "F.Cu") (net 1))
+  (segment (start 52.5 160.5) (end 52.5 158.5) (width 0.8) (layer "F.Cu") (net 1))
   (segment (start 92 154.5) (end 89 154.5) (width 0.5) (layer "F.Cu") (net 1))
   (segment (start 108.5 120.5) (end 115.5 127.5) (width 0.8) (layer "F.Cu") (net 1))
@@
   (via (at 87 49.5) (size 1) (drill 0.5) (layers "F.Cu" "B.Cu") (free) (net 1))
   (via (at 115.5 150) (size 1) (drill 0.5) (layers "F.Cu" "B.Cu") (free) (net 1))
+  (via (at 52.5 160.5) (size 0.8) (drill 0.4) (layers "F.Cu" "B.Cu") (net 1))
   (via (at 91 68.5) (size 1) (drill 0.5) (layers "F.Cu" "B.Cu") (free) (net 1))
   (via (at 89 154.5) (size 0.8) (drill 0.4) (layers "F.Cu" "B.Cu") (net 1))
@@
   (via (at 110.5 150) (size 1) (drill 0.5) (layers "F.Cu" "B.Cu") (free) (net 1))
   (via (at 104.5 65.5) (size 0.8) (drill 0.4) (layers "F.Cu" "B.Cu") (net 1))
+  (via (at 125.5 39.5) (size 0.8) (drill 0.4) (layers "F.Cu" "B.Cu") (net 1))
   (via (at 113 148) (size 1) (drill 0.5) (layers "F.Cu" "B.Cu") (free) (net 1))
   (via (at 62.5 66) (size 1) (drill 0.5) (layers "F.Cu" "B.Cu") (free) (net 1))
