File: Kicad/motors/motors.kicad_pcb (KiCad board)
At the start: 2 copper layers, 80 x 140 mm, 149 parts, among them K100 9V - 1A, K201 MOTOR 1, K202 MOTOR 2, K203 MOTOR 4, K204 MOTOR 3, K301 FRONT, K302 REAR, Q100 DMP2305U, Q101 DMP2305U, Q102 STN790A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

Commit message: Up
Parts:
- IR301, IR302, IR303, IR304: footprint tronixioZZZ:OPB-610 -> tronixio:ZZ_OPB-610
- K100: footprint tronixioZZZ:CUI-PJ-002AH-SMT-TR -> tronixio:ZZ_CUI-PJ-002AH-SMT-TR
- Q301, Q302: footprint tronixioZZZ:SOT-70-6 -> tronixio:SC-70-6
- R100, R101: footprint tronixio:RESISTOR-SMD-1210 -> tronixio:RESISTOR-SMD-1206
- S100: footprint tronixioZZZ:E-SWITCH-200USPXT1A1M6RE -> tronixio:ZZ_E-SWITCH-200USPXT1A1M6RE
- TP100, TP101, TP102, TP103, TP104, TP105, TP201, TP301: footprint tronixioZZZ:HARWIN-S1751 -> tronixio:ZZ_HARWIN-S1751
- U201, U204: footprint tronixioZZZ:SOPOWER-20 -> tronixio:SOPOWER-20
Connections:
- net /Driver/BRAKE renamed /Drivers/BRAKE
- net /Driver/M1+ renamed /Drivers/M1+
- net /Driver/M1- renamed /Drivers/M1-
- net /Driver/M1_SENSE renamed /Drivers/M1_SENSE
- net /Driver/M1_SPEED renamed /Drivers/M1_SPEED
- net /Driver/M2+ renamed /Drivers/M2+
- net /Driver/M2- renamed /Drivers/M2-
- net /Driver/M2_SENSE renamed /Drivers/M2_SENSE
- net /Driver/M2_SPEED renamed /Drivers/M2_SPEED
- net /Driver/M3+ renamed /Drivers/M3+
- net /Driver/M3- renamed /Drivers/M3-
- net /Driver/M3_SENSE renamed /Drivers/M3_SENSE
- net /Driver/M3_SPEED renamed /Drivers/M3_SPEED
- net /Driver/M4+ renamed /Drivers/M4+
- net /Driver/M4- renamed /Drivers/M4-
- net /Driver/M4_SENSE renamed /Drivers/M4_SENSE
- net /Driver/M4_SPEED renamed /Drivers/M4_SPEED
- net /Driver/STOP renamed /Drivers/STOP
Other:
- outline, holes or cut-outs redrawn

Commit message: Up
Parts:
- C203, C204, C207, C208: footprint tronixioZZZ:CAPACITOR-ELECTROLYTIC-RADIAL-100-160-050 -> tronixio:ZZ_CAPACITOR-ELECTROLYTIC-RADIAL-100-160-050

Commit message: Up
Parts:
- removed G*** (x2): LOGO, tronixALL:OSHW-5MM
- added X101: SYMBOL-MISC, tronixio:OSHW-5MM, F.Cu at (66.0, 109.0)
- added X102: SYMBOL-MISC, tronixio:OSHW-5MM, B.Cu at (89.0, 110.5)
- added kibuzzard-62897416: G***, kibuzzard-62897416, B.Cu at (77.6, 36.0)
- added kibuzzard-628974BE: G***, kibuzzard-628974BE, B.Cu at (100.5, 36.0)
- added kibuzzard-62897505: G***, kibuzzard-62897505, B.Cu at (77.6, 164.0)
- added kibuzzard-6289753B: G***, kibuzzard-6289753B, B.Cu at (100.5, 164.0)
- C203, C204, C207, C208: footprint tronixio:ZZ_CAPACITOR-ELECTROLYTIC-RADIAL-100-160-050 -> tronixio:CAPACITOR-ELECTROLYTIC-RADIAL-100-160-050
- IR301, IR302, IR303, IR304: footprint tronixio:ZZ_OPB-610 -> tronixio:OPB-610
- K100: footprint tronixio:ZZ_CUI-PJ-002AH-SMT-TR -> tronixio:CUI-PJ-002AH-SMT-TR
- S100: footprint tronixio:ZZ_E-SWITCH-200USPXT1A1M6RE -> tronixio:E-SWITCH-200USPXT1A1M6RE
- TP100, TP101, TP102, TP103, TP104, TP105, TP201, TP301: footprint tronixio:ZZ_HARWIN-S1751 -> tronixio:HARWIN-S1751
- moved S100 0.25 mm to (62.5, 164.8)
Connections:
- S100 pad 4: (no net) -> unconnected-(S100-Pad4)
Routing:
- net VIN: track 392.3 -> 383.6 mm, vias 19 -> 35
- net GND: track 177.2 -> 174.9 mm, vias 61 -> 85
- net /Drivers/BRAKE: track 211.8 -> 211.1 mm
- net Net-(Q101-G): track 91.1 -> 90.4 mm
Other:
- board text added: "202301 - Rev.A"
- board text added: "TCAR Motor Board L298P - Rev.A - (01/2023) - Scale 100%"
- board text removed: "202201 - Rev.A"
- board text removed: "GND"
- board text removed: "TCAR Motor Board L298P - Rev.A - (01/2022) - Scale 100%"
- board text removed: "VIN"
