File: Kicad/motors/driver.kicad_sch (KiCad schematic)
At the start: 60 parts, among them IC201 L298P, IC202 SN74LVC1G19, IC203 SN74LVC1G19, IC204 L298P, IC205 SN74LVC1G19, IC206 SN74LVC1G19, IC207 LM3480-50, K201 MOTOR 1, K202 MOTOR 2, K203 MOTOR 4, K204 MOTOR 3

Commit message: Update
Other:
- moved on the sheet: R211
Changed lines of the file:
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@@
     (stroke (width 0) (type solid) (color 0 0 0 0))
   )
-  (wire (pts (xy 66.04 86.36) (xy 73.66 86.36))
+  (wire (pts (xy 63.5 86.36) (xy 73.66 86.36))
     (stroke (width 0) (type default) (color 0 0 0 0))
   )
@@
     (stroke (width 0) (type solid) (color 0 0 0 0))
   )
-  (wire (pts (xy 66.04 124.46) (xy 77.47 124.46))
+  (wire (pts (xy 63.5 124.46) (xy 77.47 124.46))
     (stroke (width 0) (type solid) (color 0 0 0 0))
   )
@@
     (stroke (width 0) (type solid) (color 0 0 0 0))
   )
-  (wire (pts (xy 66.04 91.44) (xy 71.12 91.44))
+  (wire (pts (xy 63.5 91.44) (xy 71.12 91.44))
     (stroke (width 0) (type default) (color 0 0 0 0))
   )
@@
     (stroke (width 0) (type solid) (color 0 0 0 0))
   )
-  (wire (pts (xy 66.04 114.3) (xy 77.47 114.3))
+  (wire (pts (xy 63.5 114.3) (xy 77.47 114.3))
     (stroke (width 0) (type solid) (color 0 0 0 0))
   )
@@
   )
   (wire (pts (xy 73.66 116.84) (xy 77.47 116.84))
-    (stroke (width 0) (type solid) (color 0 0 0 0))
-  )
-  (wire (pts (xy 63.5 175.26) (xy 63.5 177.8))
     (stroke (width 0) (type solid) (color 0 0 0 0))
   )
@@
     (effects (font (size 1.27 1.27)) (justify left))
   )
-  (hierarchical_label "M3_SPEED" (shape input) (at 66.04 124.46 180)
+  (hierarchical_label "M3_SPEED" (shape input) (at 63.5 124.46 180)
     (effects (font (size 1.27 1.27)) (justify right))
   )
-  (hierarchical_label "M4_SPEED" (shape input) (at 66.04 114.3 180)
+  (hierarchical_label "M4_SPEED" (shape input) (at 63.5 114.3 180)
     (effects (font (size 1.27 1.27)) (justify right))
   )
@@
     (effects (font (size 1.27 1.27)) (justify left))
   )
-  (hierarchical_label "STOP" (shape input) (at 66.04 91.44 180)
+  (hierarchical_label "STOP" (shape input) (at 63.5 91.44 180)
     (effects (font (size 1.27 1.27)) (justify right))
   )
-  (hierarchical_label "BRAKE" (shape input) (at 66.04 86.36 180)
+  (hierarchical_label "BRAKE" (shape input) (at 63.5 86.36 180)
     (effects (font (size 1.27 1.27)) (justify right))
   )
@@
     (pin "2")
   )
-  (symbol (lib_id "tronixio:POWER-+5V") (at 63.5 165.1 0) (unit 1)
-    (in_bom yes) (on_board yes)
-    (property "Reference" "#PWR0237" (id 0) (at 63.5 175.26 0)
-      (effects (font (size 1 1)) hide)
-    )
-    (property "Value" "POWER-+5V" (id 1) (at 63.5 177.8 0)
-      (effects (font (size 1 1)) hide)
-    )
-    (property "Footprint" "" (id 2) (at 63.5 165.1 0)
-      (effects (font (size 1 1)) hide)
-    )
-    (property "Datasheet" "" (id 3) (at 63.5 165.1 0)
-      (effects (font (size 1 1)) hide)
-    )
-    (property "Name" "+5V" (id 4) (at 63.5 160.02 0)
+  (symbol (lib_id "tronixio:POWER-+5V") (at 63.5 167.64 0) (unit 1)
+    (in_bom yes) (on_board yes)
+    (property "Reference" "#PWR0237" (id 0) (at 63.5 177.8 0)
+      (effects (font (size 1 1)) hide)
+    )
+    (property "Value" "POWER-+5V" (id 1) (at 63.5 180.34 0)
+      (effects (font (size 1 1)) hide)
+    )
+    (property "Footprint" "" (id 2) (at 63.5 167.64 0)
+      (effects (font (size 1 1)) hide)
+    )
+    (property "Datasheet" "" (id 3) (at 63.5 167.64 0)
+      (effects (font (size 1 1)) hide)
+    )
+    (property "Name" "+5V" (id 4) (at 63.5 162.56 0)
       (effects (font (size 1.15 1.15)))
     )
@@
   (symbol (lib_id "tronixio:C-1206") (at 121.92 177.8 0) (unit 1)
     (in_bom yes) (on_board yes)
-    (property "Reference" "C210" (id 0) (at 121.92 175.26 0)
-      (effects (font (size 1.15 1.15)) (justify left))
-    )
-    (property "Value" "100n" (id 1) (at 121.92 180.34 0)
+    (property "Reference" "C210" (id 0) (at 122.555 175.26 0)
+      (effects (font (size 1.15 1.15)) (justify left))
+    )
+    (property "Value" "100n" (id 1) (at 122.555 180.34 0)
       (effects (font (size 1.15 1.15)) (justify left))
     )
@@
   (symbol (lib_id "tronixio:C-1206") (at 99.06 177.8 0) (unit 1)
     (in_bom yes) (on_board yes)
-    (property "Reference" "C209" (id 0) (at 99.06 175.26 0)
-      (effects (font (size 1.15 1.15)) (justify left))
-    )
-    (property "Value" "100n" (id 1) (at 99.06 180.34 0)
+    (property "Reference" "C209" (id 0) (at 99.695 175.26 0)
+      (effects (font (size 1.15 1.15)) (justify left))
+    )
+    (property "Value" "100n" (id 1) (at 99.695 180.34 0)
       (effects (font (size 1.15 1.15)) (justify left))
     )
@@
     (pin "2")
   )
-  (symbol (lib_id "tronixio:R-1206") (at 63.5 170.18 0) (unit 1)
-    (in_bom yes) (on_board yes)
-    (property "Reference" "R211" (id 0) (at 64.135 166.37 0)
-      (effects (font (size 1.15 1.15)) (justify left))
-    )
-    (property "Value" "12K" (id 1) (at 63.5 170.18 90)
-      (effects (font (size 1.15 1.15)))
-    )
-    (property "Footprint" "tronixio:RESISTOR-1206" (id 2) (at 63.5 182.88 0)
-      (effects (font (size 1 1)) hide)
-    )
-    (property "Datasheet" "" (id 3) (at 63.5 170.18 0)
-      (effects (font (size 1 1)) hide)
-    )
+  (symbol (lib_id "tronixio:R-1206") (at 63.5 172.72 0) (unit 1)
+    (in_bom yes) (on_board yes)
+    (property "Reference" "R211" (id 0) (at 64.135 168.91 0)
+      (effects (font (size 1.15 1.15)) (justify left))
+    )
+    (property "Value" "12K" (id 1) (at 63.5 172.72 90)
+      (effects (font (size 1.15 1.15)))
+    )
+    (property "Footprint" "tronixio:RESISTOR-1206" (id 2) (at 63.5 185.42 0)
+      (effects (font (size 1 1)) hide)
+    )
+    (property "Datasheet" "" (id 3) (at 63.5 172.72 0)
+      (effects (font (size 1 1)) hide)
+    )

Commit message: Update Motor
Parts:
- C203, C204, C207, C208: footprint tronixio:zzzCAPACITOR-ELECTROLYTIC-RADIAL-100-160-050 -> (none); MOUSER UVZ1V471MPD -> (none); Mouser (none) -> UVZ1V471MPD
- D201, D202, D203, D204, D205, D206, D207, D208, D210, D211, D212, D213, D214, D215, D216: symbol tronixio:PMEG3030 -> tronixio:NEXPERIA-PMEG3030; MOUSER 771-PMEG3030EP115 -> (none); Mouser (none) -> 771-PMEG3030EP115; Name (none) -> PMEG3030
- D209: value PMEG3030 -> (none); symbol tronixio:PMEG3030 -> tronixio:NEXPERIA-PMEG3030; MOUSER 771-PMEG3030EP115 -> (none); Mouser (none) -> 771-PMEG3030EP115; Name (none) -> PMEG3030
- IC201: value L298P -> (none); footprint tronixio:zzzSOPOWER-20 -> (none); symbol tronixio:L298P -> tronixio:ST-L298P-SOPOWER; MOUSER 511-L298P-TR -> (none); Mouser (none) -> 511-L298P-TR; Name (none) -> L298P
- IC202, IC203, IC205, IC206: symbol tronixio:SN74LVC1G19-SOT -> tronixio:TI-SN74LVC1G19-SOT; MOUSER 595-SN74LVC1G19DBVR -> (none); Mouser (none) -> 595-SN74LVC1G19DBVR; Name (none) -> SN74LVC1G19
- IC204: footprint tronixio:zzzSOPOWER-20 -> (none); symbol tronixio:L298P -> tronixio:ST-L298P-SOPOWER; MOUSER 511-L298P-TR -> (none); Mouser (none) -> 511-L298P-TR; Name (none) -> L298P
- IC207: value LM3480-50 -> (none); symbol tronixio:LM3480-50-SOT -> tronixio:TI-LM3480-50-SOT; MOUSER 926-LM3480IM35.0NOPB -> (none); Mouser (none) -> 926-LM3480IM35.0NOPB; Name (none) -> LM3480-50
- K201, K202, K203, K204: MOUSER 490-TB006-508-02BE -> (none); Mouser (none) -> 490-TB006-508-02BE
- LED201, LED202, LED203, LED204, LED205, LED206, LED207, LED208, LED209: MOUSER 604-APT3216LSECKJ3RV -> (none); Mouser (none) -> 604-APT3216LSECKJ3RV
- R208: footprint tronixio:RESISTOR-1206 -> tronixio:RESISTOR-1210
- TP201: footprint tronixio:zzzHARWIN-S1751 -> (none); MOUSER 855-S1751-46 -> (none); Mouser (none) -> 855-S1751-46

Commit message: Update
Parts:
- C203, C204, C207, C208: footprint (none) -> tronixio:zzzCAPACITOR-ELECTROLYTIC-RADIAL-100-160-050
- D201, D202, D203, D204, D205, D206, D207, D208, D210, D211, D212, D213, D214, D215, D216: value PMEG3030 -> NEXPERIA-PMEG3030
- D209: value (none) -> NEXPERIA-PMEG3030
- IC201: value (none) -> L298P; footprint (none) -> tronixio:zzzSOPOWER-20
- IC204: footprint (none) -> tronixio:zzzSOPOWER-20
- IC207: value (none) -> LM3480-50
- LED201, LED202, LED203, LED204, LED205, LED206, LED207, LED208: value Red -> LED-1206-RED; Name (none) -> Red
- LED209: value +5V -> LED-1206-RED; Name (none) -> Red
- TP201: footprint (none) -> tronixio:HARWIN-S1751; Name (none) -> GND

Commit message: Update
Parts:
- TP201: footprint tronixio:HARWIN-S1751 -> tronixio:zzzHARWIN-S1751; Name GND -> (none)
Changed lines of the file:
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@@
       (effects (font (size 1 1)) hide)
     )
-    (property "Footprint" "tronixio:HARWIN-S1751" (id 2) (at 53.34 177.8 0)
+    (property "Footprint" "tronixio:zzzHARWIN-S1751" (id 2) (at 53.34 177.8 0)
       (effects (font (size 1 1)) hide)
     )
@@
       (effects (font (size 1 1)) hide)
     )
-    (property "Name" "GND" (id 5) (at 53.34 162.56 0)
-      (effects (font (size 1.15 1.15)))
-    )
     (pin "1")
