File: Kicad/motors/driver.kicad_sch (KiCad schematic)
At the start: 60 parts, among them IC201 L298P, IC202 SN74LVC1G19, IC203 SN74LVC1G19, IC204 L298P, IC205 SN74LVC1G19, IC206 SN74LVC1G19, IC207 LM3480-50, K201 MOTOR 1, K202 MOTOR 2, K203 MOTOR 4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

Commit message: Update
Other:
- moved on the sheet: C201, C202, C203, C204, C205, C206, C207, C208, D201, D202, D203, D204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

Commit message: Update
Parts:
- C201, C202, C205, C206, C209, C210: footprint tronixio:CAPACITOR-1206 -> tronixio:CAPACITOR-SMD-1206; symbol tronixio:C-1206 -> tronixio:CAPACITOR-1206-100N; Mouser (none) -> 80-C1206C104M5R; Name (none) -> CAPACITOR-1206-100N; Tolerance (none) -> 20%; Voltage (none) -> 50V
- C203, C204, C207, C208: value UVZ-470U-35V -> 470µ/35V; footprint tronixio:zzzCAPACITOR-ELECTROLYTIC-RADIAL-100-160-050 -> tronixioZZZ:CAPACITOR-ELECTROLYTIC-RADIAL-100-160-050; symbol tronixio:UVZ-470U-35V -> tronixio:NICHICON-UVZ-470U-35V; Name 470µ/35V -> NICHICON-UVZ-470U-35V; Tolerance (none) -> 20%; Voltage (none) -> 35V
- C211, C212: footprint tronixio:CAPACITOR-1206 -> tronixio:CAPACITOR-SMD-1206; symbol tronixio:C-1206 -> tronixio:CAPACITOR-1206-1U; Mouser (none) -> C1206C105M5RACTU; Name (none) -> CAPACITOR-1206-1U; Tolerance (none) -> 20%; Voltage (none) -> 50V
- D201, D202, D203, D204, D205, D206, D207, D208, D209, D210, D211, D212, D213, D214, D215, D216: value NEXPERIA-PMEG3030 -> PMEG3030; Name PMEG3030 -> NEXPERIA-PMEG3030
- K201, K202, K203, K204: Name (none) -> CUI-TB006-508-02BE
- LED201, LED202, LED203, LED204, LED205, LED206, LED207, LED208: value LED-1206-RED -> KINGBRIGHT-LED-1206-ORANGE; footprint tronixio:LED-1206 -> tronixio:LED-SMD-1206; symbol tronixio:LED-1206-RED -> tronixio:KINGBRIGHT-LED-1206-RED; Name Red -> KINGBRIGHT-LED-1206-RED
- LED209: value LED-1206-RED -> +5V; footprint tronixio:LED-1206 -> tronixio:LED-SMD-1206; symbol tronixio:LED-1206-RED -> tronixio:KINGBRIGHT-LED-1206-RED; Name Red -> KINGBRIGHT-LED-1206-RED
- R201, R202, R203, R206, R207: footprint tronixio:RESISTOR-1206 -> tronixio:RESISTOR-SMD-1206; symbol tronixio:R-1206 -> tronixio:RESISTOR-1206-10K; Mouser (none) -> 660-RK73B2BTTDD103J; Name (none) -> RESISTOR-1206-10K; Tolerance (none) -> 5%
- R204, R205, R209, R210: footprint tronixio:RESISTOR-1210 -> tronixio:RESISTOR-SMD-1210; symbol tronixio:R-1210 -> tronixio:RESISTOR-1210-0R5; Mouser (none) -> 660-SR732ETTDR499F; Name (none) -> RESISTOR-1210-0R5; Tolerance (none) -> 1%
- R208: footprint tronixio:RESISTOR-1210 -> tronixio:RESISTOR-SMD-1206; symbol tronixio:R-1210 -> tronixio:RESISTOR-1206-10K; Mouser (none) -> 660-RK73B2BTTDD103J; Name (none) -> RESISTOR-1206-10K; Tolerance (none) -> 5%
- R211: footprint tronixio:RESISTOR-1206 -> tronixio:RESISTOR-SMD-1206; symbol tronixio:R-1206 -> tronixio:RESISTOR-1206-12K; Mouser (none) -> 660-RK73B2BTTD123J; Name (none) -> RESISTOR-1206-12K; Tolerance (none) -> 5%
- TP201: footprint tronixio:zzzHARWIN-S1751 -> tronixioZZZ:HARWIN-S1751; Name (none) -> HARWIN-S1751
- U201: renamed from IC201; footprint tronixio:zzzSOPOWER-20 -> tronixioZZZ:SOPOWER-20; Name L298P -> ST-L298P-SOPOWER
- U202: renamed from IC202; Name SN74LVC1G19 -> TI-SN74LVC1G19-SOT
- U203: renamed from IC203; Name SN74LVC1G19 -> TI-SN74LVC1G19-SOT
- U204: renamed from IC204; footprint tronixio:zzzSOPOWER-20 -> tronixioZZZ:SOPOWER-20; Name L298P -> ST-L298P-SOPOWER
- U205: renamed from IC205; Name SN74LVC1G19 -> TI-SN74LVC1G19-SOT
- U206: renamed from IC206; Name SN74LVC1G19 -> TI-SN74LVC1G19-SOT
- U207: renamed from IC207; symbol tronixio:TI-LM3480-50-SOT -> tronixio:TI-LM3480-50-SOT-23; Name LM3480-50 -> TI-LM3480-50-SOT-23
Other:
- moved on the sheet: C209, C210, R201, R208, U202A, U202B, U203A, U203B, U205A, U205B, U206A, U206B

Commit message: Update
Changed lines of the file:
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@@
     (pin "2")
   )
-  (symbol (lib_name "KINGBRIGHT-LED-1206-RED_7") (lib_id "tronixio:KINGBRIGHT-LED-1206-RED") (at 177.8 76.2 90) (unit 1)
+  (symbol (lib_id "tronixio:KINGBRIGHT-LED-1206-RED") (at 177.8 76.2 90) (unit 1)
     (in_bom yes) (on_board yes)
     (property "Reference" "LED203" (id 0) (at 176.53 74.295 0)
@@
     (pin "1")
   )
-  (symbol (lib_name "KINGBRIGHT-LED-1206-RED_8") (lib_id "tronixio:KINGBRIGHT-LED-1206-RED") (at 182.88 76.2 270) (unit 1)
+  (symbol (lib_id "tronixio:KINGBRIGHT-LED-1206-RED") (at 182.88 76.2 270) (unit 1)
     (in_bom yes) (on_board yes)
     (property "Reference" "LED204" (id 0) (at 184.15 74.295 0)
@@
     (pin "1")
   )
-  (symbol (lib_name "RESISTOR-1206-10K_5") (lib_id "tronixio:RESISTOR-1206-10K") (at 73.66 149.86 0) (unit 1)
+  (symbol (lib_id "tronixio:RESISTOR-1206-10K") (at 73.66 149.86 0) (unit 1)
     (in_bom yes) (on_board yes)
     (property "Reference" "R208" (id 0) (at 73.025 146.05 0)
@@
     (pin "2")
   )
-  (symbol (lib_name "CAPACITOR-1206-100N_4") (lib_id "tronixio:CAPACITOR-1206-100N") (at 93.98 78.74 0) (unit 1)
+  (symbol (lib_id "tronixio:CAPACITOR-1206-100N") (at 93.98 78.74 0) (unit 1)
     (in_bom yes) (on_board yes)
     (property "Reference" "C201" (id 0) (at 93.345 76.2 0)
@@
     (pin "1")
   )
-  (symbol (lib_name "KINGBRIGHT-LED-1206-RED_1") (lib_id "tronixio:KINGBRIGHT-LED-1206-RED") (at 182.88 101.6 270) (mirror x) (unit 1)
+  (symbol (lib_id "tronixio:KINGBRIGHT-LED-1206-RED") (at 182.88 101.6 270) (mirror x) (unit 1)
     (in_bom yes) (on_board yes)
     (property "Reference" "LED206" (id 0) (at 184.15 103.505 0)
@@
     (pin "2")
   )
-  (symbol (lib_name "CAPACITOR-1206-1U_1") (lib_id "tronixio:CAPACITOR-1206-1U") (at 25.4 180.34 0) (unit 1)
+  (symbol (lib_id "tronixio:CAPACITOR-1206-1U") (at 25.4 180.34 0) (unit 1)
     (in_bom yes) (on_board yes)
     (property "Reference" "C211" (id 0) (at 24.765 177.8 0)
@@
     (pin "2")
   )
-  (symbol (lib_name "CAPACITOR-1206-100N_2") (lib_id "tronixio:CAPACITOR-1206-100N") (at 152.4 149.86 0) (unit 1)
+  (symbol (lib_id "tronixio:CAPACITOR-1206-100N") (at 152.4 149.86 0) (unit 1)
     (in_bom yes) (on_board yes)
     (property "Reference" "C206" (id 0) (at 153.035 147.32 0)
@@
     (pin "2")
   )
-  (symbol (lib_id "tronixio:TI-SN74LVC1G19-SOT") (at 81.28 114.3 0) (unit 1)
+  (symbol (lib_name "TI-SN74LVC1G19-SOT_2") (lib_id "tronixio:TI-SN74LVC1G19-SOT") (at 81.28 114.3 0) (unit 1)
     (in_bom yes) (on_board yes)
     (property "Reference" "U205" (id 0) (at 85.09 109.22 0)
@@
     (pin "2")
   )
-  (symbol (lib_id "tronixio:TI-SN74LVC1G19-SOT") (at 81.28 124.46 0) (unit 1)
+  (symbol (lib_name "TI-SN74LVC1G19-SOT_3") (lib_id "tronixio:TI-SN74LVC1G19-SOT") (at 81.28 124.46 0) (unit 1)
     (in_bom yes) (on_board yes)
     (property "Reference" "U206" (id 0) (at 85.09 130.81 0)
@@
     (pin "1")
   )
-  (symbol (lib_name "KINGBRIGHT-LED-1206-RED_3") (lib_id "tronixio:KINGBRIGHT-LED-1206-RED") (at 182.88 147.32 270) (unit 1)
+  (symbol (lib_id "tronixio:KINGBRIGHT-LED-1206-RED") (at 182.88 147.32 270) (unit 1)
     (in_bom yes) (on_board yes)
     (property "Reference" "LED208" (id 0) (at 184.15 145.415 0)
@@
     (pin "2")
   )
-  (symbol (lib_id "tronixio:TI-SN74LVC1G19-SOT") (at 81.28 53.34 0) (unit 1)
+  (symbol (lib_name "TI-SN74LVC1G19-SOT_6") (lib_id "tronixio:TI-SN74LVC1G19-SOT") (at 81.28 53.34 0) (unit 1)
     (in_bom yes) (on_board yes)
     (property "Reference" "U203" (id 0) (at 85.09 59.69 0)
@@
     (pin "2")
   )
-  (symbol (lib_id "tronixio:TI-SN74LVC1G19-SOT") (at 132.08 177.8 0) (unit 2)
+  (symbol (lib_name "TI-SN74LVC1G19-SOT_1") (lib_id "tronixio:TI-SN74LVC1G19-SOT") (at 132.08 177.8 0) (unit 2)
     (in_bom yes) (on_board yes)
     (property "Reference" "U206" (id 0) (at 132.08 177.8 0)
@@
     (pin "1")
   )
-  (symbol (lib_name "KINGBRIGHT-LED-1206-RED_5") (lib_id "tronixio:KINGBRIGHT-LED-1206-RED") (at 177.8 30.48 90) (mirror x) (unit 1)
+  (symbol (lib_id "tronixio:KINGBRIGHT-LED-1206-RED") (at 177.8 30.48 90) (mirror x) (unit 1)
     (in_bom yes) (on_board yes)
     (property "Reference" "LED201" (id 0) (at 176.53 32.385 0)
@@
     (pin "5")
   )
-  (symbol (lib_name "RESISTOR-1210-0R5_3") (lib_id "tronixio:RESISTOR-1210-0R5") (at 134.62 149.86 0) (unit 1)
+  (symbol (lib_id "tronixio:RESISTOR-1210-0R5") (at 134.62 149.86 0) (unit 1)
     (in_bom yes) (on_board yes)
     (property "Reference" "R210" (id 0) (at 134.62 146.05 0)
@@
     (pin "1")
   )
-  (symbol (lib_name "RESISTOR-1206-10K_2") (lib_id "tronixio:RESISTOR-1206-10K") (at 180.34 137.16 0) (unit 1)
+  (symbol (lib_id "tronixio:RESISTOR-1206-10K") (at 180.34 137.16 0) (unit 1)
     (in_bom yes) (on_board yes)
     (property "Reference" "R207" (id 0) (at 180.975 133.35 0)
@@
     (pin "2")
   )
-  (symbol (lib_name "RESISTOR-1206-10K_3") (lib_id "tronixio:RESISTOR-1206-10K") (at 180.34 40.64 0) (unit 1)
+  (symbol (lib_id "tronixio:RESISTOR-1206-10K") (at 180.34 40.64 0) (unit 1)
     (in_bom yes) (on_board yes)
     (property "Reference" "R202" (id 0) (at 180.975 44.45 0)
@@
     (pin "2")
   )
-  (symbol (lib_id "tronixio:TI-SN74LVC1G19-SOT") (at 93.98 177.8 0) (unit 2)
+  (symbol (lib_name "TI-SN74LVC1G19-SOT_4") (lib_id "tronixio:TI-SN74LVC1G19-SOT") (at 93.98 177.8 0) (unit 2)
     (in_bom yes) (on_board yes)
     (property "Reference" "U202" (id 0) (at 93.98 177.8 0)
@@
     (pin "1")
   )
-  (symbol (lib_name "CAPACITOR-1206-100N_3") (lib_id "tronixio:CAPACITOR-1206-100N") (at 93.98 149.86 0) (unit 1)
+  (symbol (lib_id "tronixio:CAPACITOR-1206-100N") (at 93.98 149.86 0) (unit 1)
     (in_bom yes) (on_board yes)
     (property "Reference" "C205" (id 0) (at 93.345 147.32 0)
@@
     (pin "1")
   )
-  (symbol (lib_name "KINGBRIGHT-LED-1206-RED_2") (lib_id "tronixio:KINGBRIGHT-LED-1206-RED") (at 177.8 101.6 90) (mirror x) (unit 1)
+  (symbol (lib_id "tronixio:KINGBRIGHT-LED-1206-RED") (at 177.8 101.6 90) (mirror x) (unit 1)
     (in_bom yes) (on_board yes)
     (property "Reference" "LED205" (id 0) (at 176.53 103.505 0)
@@
     (pin "2")
   )
-  (symbol (lib_name "RESISTOR-1210-0R5_2") (lib_id "tronixio:RESISTOR-1210-0R5") (at 129.54 78.74 0) (unit 1)
+  (symbol (lib_id "tronixio:RESISTOR-1210-0R5") (at 129.54 78.74 0) (unit 1)
     (in_bom yes) (on_board yes)
     (property "Reference" "R204" (id 0) (at 129.54 74.93 0)
@@
     (pin "1")
   )
-  (symbol (lib_name "RESISTOR-1210-0R5_1") (lib_id "tronixio:RESISTOR-1210-0R5") (at 134.62 78.74 0) (unit 1)
+  (symbol (lib_id "tronixio:RESISTOR-1210-0R5") (at 134.62 78.74 0) (unit 1)
     (in_bom yes) (on_board yes)
     (property "Reference" "R205" (id 0) (at 134.62 74.93 0)
@@
     (pin "1")
   )
-  (symbol (lib_name "KINGBRIGHT-LED-1206-RED_4") (lib_id "tronixio:KINGBRIGHT-LED-1206-RED") (at 177.8 147.32 90) (unit 1)
+  (symbol (lib_id "tronixio:KINGBRIGHT-LED-1206-RED") (at 177.8 147.32 90) (unit 1)
     (in_bom yes) (on_board yes)
     (property "Reference" "LED207" (id 0) (at 176.53 145.415 0)
@@
     (pin "2")
   )
-  (symbol (lib_name "RESISTOR-1206-10K_4") (lib_id "tronixio:RESISTOR-1206-10K") (at 180.34 66.04 0) (unit 1)
+  (symbol (lib_id "tronixio:RESISTOR-1206-10K") (at 180.34 66.04 0) (unit 1)
     (in_bom yes) (on_board yes)
     (property "Reference" "R203" (id 0) (at 180.975 62.23 0)
@@
     (pin "1")
   )
-  (symbol (lib_name "KINGBRIGHT-LED-1206-RED_6") (lib_id "tronixio:KINGBRIGHT-LED-1206-RED") (at 182.88 30.48 270) (mirror x) (unit 1)
+  (symbol (lib_id "tronixio:KINGBRIGHT-LED-1206-RED") (at 182.88 30.48 270) (mirror x) (unit 1)
     (in_bom yes) (on_board yes)
     (property "Reference" "LED202" (id 0) (at 184.15 32.385 0)
@@
     (pin "3")
   )
-  (symbol (lib_id "tronixio:TI-SN74LVC1G19-SOT") (at 81.28 43.18 0) (unit 1)
+  (symbol (lib_name "TI-SN74LVC1G19-SOT_5") (lib_id "tronixio:TI-SN74LVC1G19-SOT") (at 81.28 43.18 0) (unit 1)
     (in_bom yes) (on_board yes)
     (property "Reference" "U202" (id 0) (at 85.09 38.1 0)
@@
     (pin "2")
   )
-  (symbol (lib_name "CAPACITOR-1206-100N_1") (lib_id "tronixio:CAPACITOR-1206-100N") (at 152.4 78.74 0) (unit 1)
+  (symbol (lib_id "tronixio:CAPACITOR-1206-100N") (at 152.4 78.74 0) (unit 1)
     (in_bom yes) (on_board yes)
     (property "Reference" "C202" (id 0) (at 153.035 76.2 0)
@@
     (pin "1")
   )
-  (symbol (lib_id "tronixio:TI-SN74LVC1G19-SOT") (at 116.84 177.8 0) (unit 2)
+  (symbol (lib_name "TI-SN74LVC1G19-SOT_7") (lib_id "tronixio:TI-SN74LVC1G19-SOT") (at 116.84 177.8 0) (unit 2)
     (in_bom yes) (on_board yes)
     (property "Reference" "U205" (id 0) (at 116.84 177.8 0)
@@
     (pin "5")
   )
-  (symbol (lib_name "CAPACITOR-1206-100N_5") (lib_id "tronixio:CAPACITOR-1206-100N") (at 101.6 177.8 0) (unit 1)
+  (symbol (lib_id "tronixio:CAPACITOR-1206-100N") (at 101.6 177.8 0) (unit 1)
     (in_bom yes) (on_board yes)
     (property "Reference" "C209" (id 0) (at 102.235 175.26 0)
@@
     (pin "1")
   )
-  (symbol (lib_name "RESISTOR-1206-10K_1") (lib_id "tronixio:RESISTOR-1206-10K") (at 180.34 111.76 0) (unit 1)
+  (symbol (lib_id "tronixio:RESISTOR-1206-10K") (at 180.34 111.76 0) (unit 1)
     (in_bom yes) (on_board yes)
     (property "Reference" "R206" (id 0) (at 180.975 115.57 0)
