File: Kicad/motors/encoder.kicad_sch (KiCad schematic)
At the start: 28 parts, among them IC301 SN74LVC2G17, IC302 SN74LVC2G17, IC303 TTE-OPB610, IC304 TTE-OPB610, IC305 TTE-OPB610, IC306 TTE-OPB610, IC307 LM3480-33, K301 Front, K302 Rear, Q301 NEXPERIA-BC846BS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

Commit message: Update
Parts:
- TP301: footprint tronixio:HARWIN-S1751 -> tronixio:zzzHARWIN-S1751; Name GND -> (none)
Changed lines of the file:
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@@
       (effects (font (size 1 1)) hide)
     )
-    (property "Footprint" "tronixio:HARWIN-S1751" (id 2) (at 53.34 177.8 0)
+    (property "Footprint" "tronixio:zzzHARWIN-S1751" (id 2) (at 53.34 177.8 0)
       (effects (font (size 1 1)) hide)
     )
@@
       (effects (font (size 1 1)) hide)
     )
-    (property "Name" "GND" (id 5) (at 53.34 162.56 0)
-      (effects (font (size 1.15 1.15)))
-    )
     (pin "1")

Commit message: Update
Parts:
- C301, C303: footprint tronixio:CAPACITOR-1206 -> tronixio:CAPACITOR-SMD-1206; symbol tronixio:C-1206 -> tronixio:CAPACITOR-1206-100N; Mouser (none) -> 80-C1206C104M5R; Name (none) -> CAPACITOR-1206-100N; Tolerance (none) -> 20%; Voltage (none) -> 50V
- C302, C304, C305, C306: footprint tronixio:CAPACITOR-1206 -> tronixio:CAPACITOR-SMD-1206; symbol tronixio:C-1206 -> tronixio:CAPACITOR-1206-1U; Mouser (none) -> C1206C105M5RACTU; Name (none) -> CAPACITOR-1206-1U; Tolerance (none) -> 20%; Voltage (none) -> 50V
- IR301: renamed from IC303; value TTE-OPB610 -> OPB610; footprint tronixio:zzzOPB-610 -> tronixioZZZ:OPB-610; Name OPB610 -> TTE-OPB610
- IR302: renamed from IC304; value TTE-OPB610 -> OPB610; footprint tronixio:zzzOPB-610 -> tronixioZZZ:OPB-610; Name OPB610 -> TTE-OPB610
- IR303: renamed from IC305; value TTE-OPB610 -> OPB610; footprint tronixio:zzzOPB-610 -> tronixioZZZ:OPB-610; Name OPB610 -> TTE-OPB610
- IR304: renamed from IC306; value TTE-OPB610 -> OPB610; footprint tronixio:zzzOPB-610 -> tronixioZZZ:OPB-610; Name OPB610 -> TTE-OPB610
- K301: value Front -> FRONT; footprint tronixio:zzHARWIN-M20-782104x -> tronixio:HARWIN-M20-782104x; Name (none) -> HARWIN-254-F-1X10-VERTICAL
- K302: value Rear -> REAR; footprint tronixio:zzHARWIN-M20-782104x -> tronixio:HARWIN-M20-782104x; Name (none) -> HARWIN-254-F-1X10-VERTICAL
- LED301: value LED-1206-RED -> +3V3; footprint tronixio:LED-1206 -> tronixio:LED-SMD-1206; symbol tronixio:LED-1206-RED -> tronixio:KINGBRIGHT-LED-1206-RED; Name Red -> KINGBRIGHT-LED-1206-RED
- Q301, Q302: value NEXPERIA-BC846BS -> BC846BS; footprint tronixio:zzzSOT-70-6 -> tronixioZZZ:SOT-70-6; Name BC846BS -> NEXPERIA-BC846BS
- R301, R302, R303, R304: footprint tronixio:RESISTOR-1206 -> tronixio:RESISTOR-SMD-1206; symbol tronixio:R-1206 -> tronixio:RESISTOR-1206-10K; Mouser (none) -> 660-RK73B2BTTDD103J; Name (none) -> RESISTOR-1206-10K; Tolerance (none) -> 5%
- R305, R306: footprint tronixio:RESISTOR-1206 -> tronixio:RESISTOR-SMD-1206; symbol tronixio:R-1206 -> tronixio:RESISTOR-1206-2K2; Mouser (none) -> 660-RK73B2BTTD222J; Name (none) -> RESISTOR-1206-2K2; Tolerance (none) -> 5%
- R307, R308: footprint tronixio:RESISTOR-1206 -> tronixio:RESISTOR-SMD-1206; symbol tronixio:R-1206 -> tronixio:RESISTOR-1206-33R; Mouser (none) -> 660-RK73B2BTTDD330J; Name (none) -> RESISTOR-1206-33R; Tolerance (none) -> 5%
- R309: footprint tronixio:RESISTOR-1206 -> tronixio:RESISTOR-SMD-1206; symbol tronixio:R-1206 -> tronixio:RESISTOR-1206-6K8; Mouser (none) -> 660-RK73B2BTTDD682J; Name (none) -> RESISTOR-1206-6K8; Tolerance (none) -> 5%
- TP301: footprint tronixio:zzzHARWIN-S1751 -> tronixioZZZ:HARWIN-S1751; Name (none) -> HARWIN-S1751
- U301: renamed from IC301; Name SN74LVC2G17 -> TI-SN74LVC2G17-SOT
- U302: renamed from IC302; Name SN74LVC2G17 -> TI-SN74LVC2G17-SOT
- U303: renamed from IC307; symbol tronixio:TI-LM3480-33-SOT -> tronixio:TI-LM3480-33-SOT-23; Name LM3480-33 -> TI-LM3480-33-SOT-23

Commit message: Update
Changed lines of the file:
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@@
     (effects (font (size 1.27 1.27)) (justify left))
   )
-  (symbol (lib_name "RESISTOR-1206-33R_1") (lib_id "tronixio:RESISTOR-1206-33R") (at 91.44 119.38 0) (unit 1)
+  (symbol (lib_id "tronixio:RESISTOR-1206-33R") (at 91.44 119.38 0) (unit 1)
     (in_bom yes) (on_board yes)
     (property "Reference" "R307" (id 0) (at 91.44 115.57 0)
@@
     (pin "2")
   )
-  (symbol (lib_name "RESISTOR-1206-10K_1") (lib_id "tronixio:RESISTOR-1206-10K") (at 96.52 43.18 0) (unit 1)
+  (symbol (lib_id "tronixio:RESISTOR-1206-10K") (at 96.52 43.18 0) (unit 1)
     (in_bom yes) (on_board yes)
     (property "Reference" "R301" (id 0) (at 97.155 39.37 0)
@@
     (pin "2")
   )
-  (symbol (lib_name "CAPACITOR-1206-100N_1") (lib_id "tronixio:CAPACITOR-1206-100N") (at 101.6 177.8 0) (unit 1)
+  (symbol (lib_id "tronixio:CAPACITOR-1206-100N") (at 101.6 177.8 0) (unit 1)
     (in_bom yes) (on_board yes)
     (property "Reference" "C301" (id 0) (at 102.235 175.26 0)
@@
     (pin "1")
   )
-  (symbol (lib_name "RESISTOR-1206-10K_2") (lib_id "tronixio:RESISTOR-1206-10K") (at 96.52 81.28 0) (unit 1)
+  (symbol (lib_id "tronixio:RESISTOR-1206-10K") (at 96.52 81.28 0) (unit 1)
     (in_bom yes) (on_board yes)
     (property "Reference" "R303" (id 0) (at 97.155 77.47 0)
@@
     (pin "2")
   )
-  (symbol (lib_name "CAPACITOR-1206-1U_1") (lib_id "tronixio:CAPACITOR-1206-1U") (at 45.72 180.34 0) (unit 1)
+  (symbol (lib_id "tronixio:CAPACITOR-1206-1U") (at 45.72 180.34 0) (unit 1)
     (in_bom yes) (on_board yes)
     (property "Reference" "C306" (id 0) (at 46.355 177.8 0)
@@
   (symbol (lib_id "tronixio:TI-SN74LVC2G17-SOT") (at 210.82 86.36 0) (unit 2)
     (in_bom yes) (on_board yes)
-    (property "Reference" "U302" (id 0) (at 210.82 82.55 0)
-      (effects (font (size 1.15 1.15)))
-    )
-    (property "Value" "SN74LVC2G17" (id 1) (at 210.82 90.17 0)
+    (property "Reference" "U302" (id 0) (at 210.82 80.01 0)
+      (effects (font (size 1.15 1.15)))
+    )
+    (property "Value" "SN74LVC2G17" (id 1) (at 210.82 82.55 0)
       (effects (font (size 1.15 1.15)))
     )
@@
   (symbol (lib_id "tronixio:TI-SN74LVC2G17-SOT") (at 109.22 48.26 0) (unit 1)
     (in_bom yes) (on_board yes)
-    (property "Reference" "U301" (id 0) (at 109.22 44.45 0)
-      (effects (font (size 1.15 1.15)))
-    )
-    (property "Value" "SN74LVC2G17" (id 1) (at 109.22 52.07 0)
+    (property "Reference" "U301" (id 0) (at 109.22 41.91 0)
+      (effects (font (size 1.15 1.15)))
+    )
+    (property "Value" "SN74LVC2G17" (id 1) (at 109.22 44.45 0)
       (effects (font (size 1.15 1.15)))
     )
@@
     (pin "1")
   )
-  (symbol (lib_name "RESISTOR-1206-2K2_1") (lib_id "tronixio:RESISTOR-1206-2K2") (at 76.2 104.14 90) (unit 1)
+  (symbol (lib_id "tronixio:RESISTOR-1206-2K2") (at 76.2 104.14 90) (unit 1)
     (in_bom yes) (on_board yes)
     (property "Reference" "R305" (id 0) (at 78.74 101.6 90)
@@
   (symbol (lib_id "tronixio:TI-SN74LVC2G17-SOT") (at 109.22 86.36 0) (unit 2)
     (in_bom yes) (on_board yes)
-    (property "Reference" "U301" (id 0) (at 109.22 82.55 0)
-      (effects (font (size 1.15 1.15)))
-    )
-    (property "Value" "SN74LVC2G17" (id 1) (at 109.22 90.17 0)
+    (property "Reference" "U301" (id 0) (at 109.22 80.01 0)
+      (effects (font (size 1.15 1.15)))
+    )
+    (property "Value" "SN74LVC2G17" (id 1) (at 109.22 82.55 0)
       (effects (font (size 1.15 1.15)))
     )
@@
     (pin "5")
   )
-  (symbol (lib_name "CAPACITOR-1206-1U_2") (lib_id "tronixio:CAPACITOR-1206-1U") (at 25.4 180.34 0) (unit 1)
+  (symbol (lib_id "tronixio:CAPACITOR-1206-1U") (at 25.4 180.34 0) (unit 1)
     (in_bom yes) (on_board yes)
     (property "Reference" "C305" (id 0) (at 24.765 177.8 0)
@@
   (symbol (lib_id "tronixio:TI-SN74LVC2G17-SOT") (at 210.82 48.26 0) (unit 1)
     (in_bom yes) (on_board yes)
-    (property "Reference" "U302" (id 0) (at 210.82 44.45 0)
-      (effects (font (size 1.15 1.15)))
-    )
-    (property "Value" "SN74LVC2G17" (id 1) (at 210.82 52.07 0)
+    (property "Reference" "U302" (id 0) (at 210.82 41.91 0)
+      (effects (font (size 1.15 1.15)))
+    )
+    (property "Value" "SN74LVC2G17" (id 1) (at 210.82 44.45 0)
       (effects (font (size 1.15 1.15)))
     )
@@
     (pin "4")
   )
-  (symbol (lib_name "RESISTOR-1206-10K_3") (lib_id "tronixio:RESISTOR-1206-10K") (at 198.12 81.28 0) (unit 1)
+  (symbol (lib_id "tronixio:RESISTOR-1206-10K") (at 198.12 81.28 0) (unit 1)
     (in_bom yes) (on_board yes)
     (property "Reference" "R304" (id 0) (at 198.755 77.47 0)
@@
     (pin "1")
   )
-  (symbol (lib_name "CAPACITOR-1206-1U_3") (lib_id "tronixio:CAPACITOR-1206-1U") (at 132.08 177.8 0) (unit 1)
+  (symbol (lib_id "tronixio:CAPACITOR-1206-1U") (at 132.08 177.8 0) (unit 1)
     (in_bom yes) (on_board yes)
     (property "Reference" "C304" (id 0) (at 132.715 175.26 0)
