File: Kicad/motors/motors.kicad_sch (KiCad schematic)
At the start: 47 parts, among them IC100 BQ2057W, K100 Charger, Q100 DIODESINC-DMP2305U-SOT-23, Q101 DIODESINC-DMP2305U-SOT-23, Q102 ST-STN790A

Commit message: Update
Parts:
- K100: footprint tronixio:CUI-PJ-002AH-SMT-TR -> tronixio:zzzCUI-PJ-002AH-SMT-TR
- TP100: footprint tronixio:HARWIN-S1751 -> tronixio:zzzHARWIN-S1751; Name VBAT -> (none)
- TP101: footprint tronixio:HARWIN-S1751 -> tronixio:zzzHARWIN-S1751; Name VIN -> (none)
- TP102, TP103: footprint tronixio:HARWIN-S1751 -> tronixio:zzzHARWIN-S1751; Name GND -> (none)
- TP104, TP105: Name GND -> (none)
Changed lines of the file:
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@@
     )
   )
-  (symbol (lib_id "tronixio:KEYSTONE-2000-3") (at 106.68 104.14 0) (unit 1)
-    (in_bom yes) (on_board yes)
-    (property "Reference" "TP105" (id 0) (at 106.68 96.52 0)
+  (symbol (lib_name "KEYSTONE-2000-3_1") (lib_id "tronixio:KEYSTONE-2000-3") (at 106.68 104.14 0) (unit 1)
+    (in_bom yes) (on_board yes)
+    (property "Reference" "TP105" (id 0) (at 106.68 99.06 0)
       (effects (font (size 1.15 1.15)))
     )
@@
       (effects (font (size 1 1)) hide)
     )
-    (property "Name" "GND" (id 5) (at 106.68 99.06 0)
-      (effects (font (size 1.15 1.15)))
-    )
     (pin "1")
   )
@@
     (pin "1")
   )
-  (symbol (lib_name "HARWIN-S1751_2") (lib_id "tronixio:HARWIN-S1751") (at 109.22 48.26 0) (unit 1)
-    (in_bom yes) (on_board yes)
-    (property "Reference" "TP101" (id 0) (at 109.22 40.64 0)
+  (symbol (lib_id "tronixio:HARWIN-S1751") (at 109.22 48.26 0) (unit 1)
+    (in_bom yes) (on_board yes)
+    (property "Reference" "TP101" (id 0) (at 109.22 43.18 0)
       (effects (font (size 1.15 1.15)))
     )
@@
       (effects (font (size 1 1)) hide)
     )
-    (property "Footprint" "tronixio:HARWIN-S1751" (id 2) (at 109.22 58.42 0)
+    (property "Footprint" "tronixio:zzzHARWIN-S1751" (id 2) (at 109.22 58.42 0)
       (effects (font (size 1 1)) hide)
     )
@@
     (property "Mouser" "855-S1751-46" (id 4) (at 109.22 63.5 0)
       (effects (font (size 1 1)) hide)
-    )
-    (property "Name" "VIN" (id 5) (at 109.22 43.18 0)
-      (effects (font (size 1.15 1.15)))
     )
     (pin "1")
@@
     )
   )
-  (symbol (lib_name "HARWIN-S1751_1") (lib_id "tronixio:HARWIN-S1751") (at 58.42 48.26 0) (unit 1)
-    (in_bom yes) (on_board yes)
-    (property "Reference" "TP100" (id 0) (at 58.42 40.64 0)
+  (symbol (lib_id "tronixio:HARWIN-S1751") (at 58.42 48.26 0) (unit 1)
+    (in_bom yes) (on_board yes)
+    (property "Reference" "TP100" (id 0) (at 58.42 43.18 0)
       (effects (font (size 1.15 1.15)))
     )
@@
       (effects (font (size 1 1)) hide)
     )
-    (property "Footprint" "tronixio:HARWIN-S1751" (id 2) (at 58.42 58.42 0)
+    (property "Footprint" "tronixio:zzzHARWIN-S1751" (id 2) (at 58.42 58.42 0)
       (effects (font (size 1 1)) hide)
     )
@@
     (property "Mouser" "855-S1751-46" (id 4) (at 58.42 63.5 0)
       (effects (font (size 1 1)) hide)
-    )
-    (property "Name" "VBAT" (id 5) (at 58.42 43.18 0)
-      (effects (font (size 1.15 1.15)))
     )
     (pin "1")
@@
     (pin "2")
   )
-  (symbol (lib_id "tronixio:HARWIN-S1751") (at 68.58 104.14 0) (unit 1)
-    (in_bom yes) (on_board yes)
-    (property "Reference" "TP102" (id 0) (at 68.58 96.52 0)
+  (symbol (lib_name "HARWIN-S1751_3") (lib_id "tronixio:HARWIN-S1751") (at 68.58 104.14 0) (unit 1)
+    (in_bom yes) (on_board yes)
+    (property "Reference" "TP102" (id 0) (at 68.58 99.06 0)
       (effects (font (size 1.15 1.15)))
     )
@@
       (effects (font (size 1 1)) hide)
     )
-    (property "Footprint" "tronixio:HARWIN-S1751" (id 2) (at 68.58 114.3 0)
+    (property "Footprint" "tronixio:zzzHARWIN-S1751" (id 2) (at 68.58 114.3 0)
       (effects (font (size 1 1)) hide)
     )
@@
     (property "Mouser" "855-S1751-46" (id 4) (at 68.58 119.38 0)
       (effects (font (size 1 1)) hide)
-    )
-    (property "Name" "GND" (id 5) (at 68.58 99.06 0)
-      (effects (font (size 1.15 1.15)))
     )
     (pin "1")
@@
   (symbol (lib_id "tronixio:HARWIN-S1751") (at 81.28 104.14 0) (unit 1)
     (in_bom yes) (on_board yes)
-    (property "Reference" "TP103" (id 0) (at 81.28 96.52 0)
+    (property "Reference" "TP103" (id 0) (at 81.28 99.06 0)
       (effects (font (size 1.15 1.15)))
     )
@@
       (effects (font (size 1 1)) hide)
     )
-    (property "Footprint" "tronixio:HARWIN-S1751" (id 2) (at 81.28 114.3 0)
+    (property "Footprint" "tronixio:zzzHARWIN-S1751" (id 2) (at 81.28 114.3 0)
       (effects (font (size 1 1)) hide)
     )
@@
       (effects (font (size 1 1)) hide)
     )
-    (property "Name" "GND" (id 5) (at 81.28 99.06 0)
-      (effects (font (size 1.15 1.15)))
-    )
     (pin "1")
   )
@@
   (symbol (lib_id "tronixio:KEYSTONE-2000-3") (at 93.98 104.14 0) (unit 1)
     (in_bom yes) (on_board yes)
-    (property "Reference" "TP104" (id 0) (at 93.98 96.52 0)
+    (property "Reference" "TP104" (id 0) (at 93.98 99.06 0)
       (effects (font (size 1.15 1.15)))
     )
@@
       (effects (font (size 1 1)) hide)
     )
-    (property "Name" "GND" (id 5) (at 93.98 99.06 0)
-      (effects (font (size 1.15 1.15)))
-    )
     (pin "1")
   )
@@
       (effects (font (size 1.15 1.15)))
     )
-    (property "Footprint" "tronixio:CUI-PJ-002AH-SMT-TR" (id 2) (at 152.4 63.5 0)
+    (property "Footprint" "tronixio:zzzCUI-PJ-002AH-SMT-TR" (id 2) (at 152.4 63.5 0)
       (effects (font (size 1 1)) hide)
     )
@@
     )
     (path "/e82e0d0d-31ce-41e5-8345-5d87bc746c22"
-      (reference "K100") (unit 1) (value "Charger") (footprint "tronixio:CUI-PJ-002AH-SMT-TR")
+      (reference "K100") (unit 1) (value "Charger") (footprint "tronixio:zzzCUI-PJ-002AH-SMT-TR")
     )
     (path "/6012b3a0-2f30-4458-8240-bd443182c6c0/fbf68a94-0255-4357-b0c0-377ea44b5b13"
@@
     )
     (path "/5155a1b3-f233-4b92-b6db-b2011c65f346"
-      (reference "TP100") (unit 1) (value "HARWIN-S1751") (footprint "tronixio:HARWIN-S1751")
+      (reference "TP100") (unit 1) (value "HARWIN-S1751") (footprint "tronixio:zzzHARWIN-S1751")
     )
     (path "/09047c60-b432-4721-9588-b4f0e2d1ccb7"
-      (reference "TP101") (unit 1) (value "HARWIN-S1751") (footprint "tronixio:HARWIN-S1751")
+      (reference "TP101") (unit 1) (value "HARWIN-S1751") (footprint "tronixio:zzzHARWIN-S1751")
     )
     (path "/afb03782-0df8-4682-84f7-c2174f611fc2"
-      (reference "TP102") (unit 1) (value "HARWIN-S1751") (footprint "tronixio:HARWIN-S1751")
+      (reference "TP102") (unit 1) (value "HARWIN-S1751") (footprint "tronixio:zzzHARWIN-S1751")
     )
     (path "/cbac58c1-51ae-4e10-a102-57fee0c17b41"
-      (reference "TP103") (unit 1) (value "HARWIN-S1751") (footprint "tronixio:HARWIN-S1751")
+      (reference "TP103") (unit 1) (value "HARWIN-S1751") (footprint "tronixio:zzzHARWIN-S1751")
     )
     (path "/e1b30331-46df-4996-a3a8-9222dc31cdda"
@@
     )
     (path "/6012b3a0-2f30-4458-8240-bd443182c6c0/8cb2d75e-5fa9-4af5-a5eb-dd77b950ebe4"
-      (reference "TP201") (unit 1) (value "HARWIN-S1751") (footprint "tronixio:HARWIN-S1751")
+      (reference "TP201") (unit 1) (value "HARWIN-S1751") (footprint "tronixio:zzzHARWIN-S1751")
     )
     (path "/56bd3a46-de12-45e9-9566-afec966f2cad/3998511c-92d7-47a9-a14d-03d7a4caa4e6"
-      (reference "TP301") (unit 1) (value "HARWIN-S1751") (footprint "tronixio:HARWIN-S1751")
-    )
-  )
+      (reference "TP301") (unit 1) (value "HARWIN-S1751") (footprint "tronixio:zzzHARWIN-S1751")
+    )
+  )

Commit message: Update
Parts:
- BT100: value 2x18650 -> 18650; Name (none) -> KEYSTONE-1049
- C100: footprint tronixio:CAPACITOR-1206 -> tronixio:CAPACITOR-SMD-1206; symbol tronixio:C-1206 -> tronixio:CAPACITOR-1206-100N; Mouser (none) -> 80-C1206C104M5R; Name (none) -> CAPACITOR-1206-100N; Tolerance (none) -> 20%; Voltage (none) -> 50V
- C101: footprint tronixio:CAPACITOR-1206 -> tronixio:CAPACITOR-SMD-1206; symbol tronixio:C-1206 -> tronixio:CAPACITOR-1206-1U; Mouser (none) -> C1206C105M5RACTU; Name (none) -> CAPACITOR-1206-1U; Tolerance (none) -> 20%; Voltage (none) -> 50V
- D100: value NEXPERIA-PMEG3030 -> PMEG3030; Name PMEG3030 -> NEXPERIA-PMEG3030
- H101, H102, H103, H104, H105, H106, H107, H108, H109, H110, H111, H112, H113, H114, H115, H116: value MOUNTING-HOLE-MASK-3MM -> MOUNTING-HOLE-3MM-MASK; footprint tronixio:M3-MASK -> tronixio:MOUNTING-HOLE-3MM-MASK; symbol tronixio:MOUNTING-HOLE-MASK-3MM -> tronixio:MOUNTING-HOLE-3MM-MASK
- H117, H118, H119, H120: value MOUNTING-HOLE-MASK-3MM -> MOUNTING-HOLE-3.5MM; footprint tronixio:M3.5 -> tronixio:MOUNTING-HOLE-3.5MM
- K100: value Charger -> CHARGER; footprint tronixio:zzzCUI-PJ-002AH-SMT-TR -> tronixioZZZ:CUI-PJ-002AH-SMT-TR; Name (none) -> CUI-PJ-002AH-SMT-TR
- LED100: value LED-1206-RED -> CHARGE; footprint tronixio:LED-1206 -> tronixio:LED-SMD-1206; symbol tronixio:LED-1206-RED -> tronixio:KINGBRIGHT-LED-1206-RED; Name Red -> KINGBRIGHT-LED-1206-RED
- LED101: value LED-1206-RED -> POWER; footprint tronixio:LED-1206 -> tronixio:LED-SMD-1206; symbol tronixio:LED-1206-RED -> tronixio:KINGBRIGHT-LED-1206-RED; Name Red -> KINGBRIGHT-LED-1206-RED
- Q100, Q101: value DIODESINC-DMP2305U-SOT-23 -> DMP2305U; Name DMP2305U -> DIODESINC-DMP2305U-SOT-23
- Q102: value ST-STN790A -> STN790A; symbol tronixio:ST-STN790A -> tronixio:ST-STN790A-SOT-223; Name STN90 -> ST-STN790A-SOT-223
- R100, R101: footprint tronixio:RESISTOR-1210 -> tronixio:RESISTOR-SMD-1210; symbol tronixio:R-1210 -> tronixio:RESISTOR-1210-0R1; Mouser (none) -> 660-SR732ETTER100F; Name (none) -> RESISTOR-1210-0R1; Tolerance (none) -> 1%
- R102: footprint tronixio:RESISTOR-1206 -> tronixio:RESISTOR-SMD-1206; symbol tronixio:R-1206 -> tronixio:RESISTOR-1206-1K; Mouser (none) -> 660-RK73B2BTTDD102J; Name (none) -> RESISTOR-1206-1K; Tolerance (none) -> 5%
- R103, R105: footprint tronixio:RESISTOR-1206 -> tronixio:RESISTOR-SMD-1206; symbol tronixio:R-1206 -> tronixio:RESISTOR-1206-10K; Mouser (none) -> 660-RK73B2BTTDD103J; Name (none) -> RESISTOR-1206-10K; Tolerance (none) -> 5%
- R104: footprint tronixio:RESISTOR-1206 -> tronixio:RESISTOR-SMD-1206; symbol tronixio:R-1206 -> tronixio:RESISTOR-1206-1M; Mouser (none) -> 660-RK73B2BTTDD105J; Name (none) -> RESISTOR-1206-1M; Tolerance (none) -> 5%
- R106: footprint tronixio:RESISTOR-1206 -> tronixio:RESISTOR-SMD-1206; symbol tronixio:R-1206 -> tronixio:RESISTOR-1206-36K; Mouser (none) -> 660-RK73B2BTTD363J; Name (none) -> RESISTOR-1206-36K; Tolerance (none) -> 5%
- R107: footprint tronixio:RESISTOR-1206 -> tronixio:RESISTOR-SMD-1206; symbol tronixio:R-1206 -> tronixio:RESISTOR-1206-15K; Mouser (none) -> 660-RK73B2BTTD153J; Name (none) -> RESISTOR-1206-15K; Tolerance (none) -> 5%
- S100: value On/Off -> ON/OFF; footprint tronixio:zzzE-SWITCH-200USPXT1A1M6RE -> tronixioZZZ:E-SWITCH-200USPXT1A1M6RE; Name (none) -> E-SWITCH-200USP1T1A1M6RE
- TH100: value 10K -> NTC-10K; footprint tronixio:THERMISTOR -> tronixio:THERMISTOR-SMD; Name 10K -> THERMISTOR-NTC-10K
- TP100, TP101, TP102, TP103: footprint tronixio:zzzHARWIN-S1751 -> tronixioZZZ:HARWIN-S1751; Name (none) -> HARWIN-S1751
- TP104, TP105: Name (none) -> KEYSTONE-2000-3
- U100: renamed from IC100; symbol tronixio:TI-BQ2057W -> tronixio:TI-BQ2057W-SOIC-08; Name BQ2057W -> TI-BQ2057W-SOIC
Other:
- moved on the sheet: R105

Commit message: Update
Parts:
- K100: value CHARGER -> 9V - 1A
Other:
- note removed: "9V - 1A"
- title: Power -> Motors Power
Changed lines of the file:
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@@
   (paper "A4")
   (title_block
-    (title "Power")
+    (title "Motors Power")
     (date "01/2022")
     (rev "A")
@@
     (effects (font (size 1.27 1.27)) (justify left bottom))
   )
-  (text "9V - 1A" (at 147.32 57.15 180)
-    (effects (font (size 1.27 1.27)) (justify right bottom))
-  )
   (text "*" (at 230.505 73.66 180)
     (effects (font (size 1.27 1.27)) (justify right bottom))
@@
   (symbol (lib_id "tronixio:E-SWITCH-200USP1T1A1M6RE") (at 85.09 76.2 90) (unit 1)
     (in_bom yes) (on_board yes)
-    (property "Reference" "S100" (id 0) (at 80.01 81.28 90)
-      (effects (font (size 1.15 1.15)) (justify right))
-    )
-    (property "Value" "ON/OFF" (id 1) (at 80.01 83.82 90)
-      (effects (font (size 1.15 1.15)) (justify right))
+    (property "Reference" "S100" (id 0) (at 85.09 71.12 90)
+      (effects (font (size 1.15 1.15)) (justify left))
+    )
+    (property "Value" "ON/OFF" (id 1) (at 85.09 81.28 90)
+      (effects (font (size 1.15 1.15)) (justify left))
     )
     (property "Footprint" "tronixioZZZ:E-SWITCH-200USPXT1A1M6RE" (id 2) (at 95.25 76.2 0)
@@
     (pin "1")
   )
-  (symbol (lib_name "RESISTOR-1206-10K_1") (lib_id "tronixio:RESISTOR-1206-10K") (at 228.6 53.34 0) (unit 1)
+  (symbol (lib_id "tronixio:RESISTOR-1206-10K") (at 228.6 53.34 0) (unit 1)
     (in_bom yes) (on_board yes)
     (property "Reference" "R103" (id 0) (at 229.235 49.53 0)
@@
     (pin "2")
   )
-  (symbol (lib_name "RESISTOR-1210-0R1_1") (lib_id "tronixio:RESISTOR-1210-0R1") (at 195.58 45.72 90) (unit 1)
+  (symbol (lib_id "tronixio:RESISTOR-1210-0R1") (at 195.58 45.72 90) (unit 1)
     (in_bom yes) (on_board yes)
     (property "Reference" "R101" (id 0) (at 195.58 43.18 90)
@@
       (effects (font (size 1.15 1.15)))
     )
-    (property "Value" "CHARGER" (id 1) (at 152.4 60.96 0)
+    (property "Value" "9V - 1A" (id 1) (at 152.4 60.96 0)
       (effects (font (size 1.15 1.15)))
     )
@@
     (pin "1")
   )
-  (symbol (lib_name "KINGBRIGHT-LED-1206-RED_1") (lib_id "tronixio:KINGBRIGHT-LED-1206-RED") (at 170.18 76.2 90) (unit 1)
+  (symbol (lib_id "tronixio:KINGBRIGHT-LED-1206-RED") (at 170.18 76.2 90) (unit 1)
     (in_bom yes) (on_board yes)
     (property "Reference" "LED100" (id 0) (at 169.545 73.66 90)
@@
     )
     (path "/e82e0d0d-31ce-41e5-8345-5d87bc746c22"
-      (reference "K100") (unit 1) (value "CHARGER") (footprint "tronixioZZZ:CUI-PJ-002AH-SMT-TR")
+      (reference "K100") (unit 1) (value "9V - 1A") (footprint "tronixioZZZ:CUI-PJ-002AH-SMT-TR")
     )
     (path "/6012b3a0-2f30-4458-8240-bd443182c6c0/fbf68a94-0255-4357-b0c0-377ea44b5b13"

Commit message: Update
Parts:
- TP104, TP105: footprint tronixio:KEYSTONE-2000-3 -> tronixioZZZ:HARWIN-S1751; symbol tronixio:KEYSTONE-2000-3 -> tronixio:HARWIN-S1751; Mouser 534-2000-3 -> 855-S1751-46; Name KEYSTONE-2000-3 -> HARWIN-S1751
Changed lines of the file:
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@@
     )
   )
-  (symbol (lib_id "tronixio:KEYSTONE-2000-3") (at 106.68 104.14 0) (unit 1)
+  (symbol (lib_id "tronixio:HARWIN-S1751") (at 106.68 104.14 0) (unit 1)
     (in_bom yes) (on_board yes)
     (property "Reference" "TP105" (id 0) (at 106.68 99.06 0)
@@
       (effects (font (size 1.15 1.15)) hide)
     )
-    (property "Footprint" "tronixio:KEYSTONE-2000-3" (id 2) (at 106.68 114.3 0)
-      (effects (font (size 1 1)) hide)
-    )
-    (property "Datasheet" "https://www.keyelco.com/product.cfm/product_id/3037" (id 3) (at 106.68 116.84 0)
-      (effects (font (size 1 1)) hide)
-    )
-    (property "Mouser" "534-2000-3" (id 4) (at 106.68 119.38 0)
-      (effects (font (size 1 1)) hide)
-    )
-    (property "Name" "KEYSTONE-2000-3" (id 5) (at 106.68 111.76 0)
+    (property "Footprint" "tronixioZZZ:HARWIN-S1751" (id 2) (at 106.68 114.3 0)
+      (effects (font (size 1 1)) hide)
+    )
+    (property "Datasheet" "https://www.harwin.com/products/S1751-46/" (id 3) (at 106.68 116.84 0)
+      (effects (font (size 1 1)) hide)
+    )
+    (property "Mouser" "855-S1751-46" (id 4) (at 106.68 119.38 0)
+      (effects (font (size 1 1)) hide)
+    )
+    (property "Name" "HARWIN-S1751" (id 5) (at 106.68 111.76 0)
       (effects (font (size 1 1)) hide)
     )
@@
     (pin "1")
   )
-  (symbol (lib_id "tronixio:KEYSTONE-2000-3") (at 93.98 104.14 0) (unit 1)
+  (symbol (lib_id "tronixio:HARWIN-S1751") (at 93.98 104.14 0) (unit 1)
     (in_bom yes) (on_board yes)
     (property "Reference" "TP104" (id 0) (at 93.98 99.06 0)
@@
       (effects (font (size 1.15 1.15)) hide)
     )
-    (property "Footprint" "tronixio:KEYSTONE-2000-3" (id 2) (at 93.98 114.3 0)
-      (effects (font (size 1 1)) hide)
-    )
-    (property "Datasheet" "https://www.keyelco.com/product.cfm/product_id/3037" (id 3) (at 93.98 116.84 0)
-      (effects (font (size 1 1)) hide)
-    )
-    (property "Mouser" "534-2000-3" (id 4) (at 93.98 119.38 0)
-      (effects (font (size 1 1)) hide)
-    )
-    (property "Name" "KEYSTONE-2000-3" (id 5) (at 93.98 111.76 0)
+    (property "Footprint" "tronixioZZZ:HARWIN-S1751" (id 2) (at 93.98 114.3 0)
+      (effects (font (size 1 1)) hide)
+    )
+    (property "Datasheet" "https://www.harwin.com/products/S1751-46/" (id 3) (at 93.98 116.84 0)
+      (effects (font (size 1 1)) hide)
+    )
+    (property "Mouser" "855-S1751-46" (id 4) (at 93.98 119.38 0)
+      (effects (font (size 1 1)) hide)
+    )
+    (property "Name" "HARWIN-S1751" (id 5) (at 93.98 111.76 0)
       (effects (font (size 1 1)) hide)
     )
@@
     )
     (path "/e1b30331-46df-4996-a3a8-9222dc31cdda"
-      (reference "TP104") (unit 1) (value "KEYSTONE-2000-3") (footprint "tronixio:KEYSTONE-2000-3")
+      (reference "TP104") (unit 1) (value "KEYSTONE-2000-3") (footprint "tronixioZZZ:HARWIN-S1751")
     )
     (path "/02ae7927-bb1b-4c3c-9b59-633a011c9114"
-      (reference "TP105") (unit 1) (value "KEYSTONE-2000-3") (footprint "tronixio:KEYSTONE-2000-3")
+      (reference "TP105") (unit 1) (value "KEYSTONE-2000-3") (footprint "tronixioZZZ:HARWIN-S1751")
     )
     (path "/6012b3a0-2f30-4458-8240-bd443182c6c0/8cb2d75e-5fa9-4af5-a5eb-dd77b950ebe4"

Commit message: Up
Parts:
- C100: symbol tronixio:CAPACITOR-1206-100N -> tronixio:CAPACITOR-1206-100N-10P-X7R; Mouser 80-C1206C104M5R -> 80-C1206C104K5R; Name CAPACITOR-1206-100N -> (none); Tolerance 20% -> 10%
- C101: symbol tronixio:CAPACITOR-1206-1U -> tronixio:CAPACITOR-1206-1U-10P-X7R; Mouser C1206C105M5RACTU -> 80-C1206C105K5R; Name CAPACITOR-1206-1U -> (none); Tolerance 20% -> 10%
- D100: Name NEXPERIA-PMEG3030 -> (none)
- K100: footprint tronixioZZZ:CUI-PJ-002AH-SMT-TR -> tronixio:ZZ_CUI-PJ-002AH-SMT-TR; Name CUI-PJ-002AH-SMT-TR -> (none)
- LED100, LED101: Name KINGBRIGHT-LED-1206-RED -> (none)
- Q100, Q101: symbol tronixio:DIODESINC-DMP2305U-SOT-23 -> tronixio:DIODES-DMP2305U-SOT-23; Name DIODESINC-DMP2305U-SOT-23 -> (none)
- R100, R101: footprint tronixio:RESISTOR-SMD-1210 -> tronixio:RESISTOR-SMD-1206; symbol tronixio:RESISTOR-1210-0R1 -> tronixio:RESISTOR-1206-0R1-5P; Name RESISTOR-1210-0R1 -> (none); Tolerance 1% -> 5%
- R102: symbol tronixio:RESISTOR-1206-1K -> tronixio:RESISTOR-1206-1K-5P; Name RESISTOR-1206-1K -> (none)
- R103, R105: symbol tronixio:RESISTOR-1206-10K -> tronixio:RESISTOR-1206-10K-5P; Name RESISTOR-1206-10K -> (none)
- R104: symbol tronixio:RESISTOR-1206-1M -> tronixio:RESISTOR-1206-1M-5P; Name RESISTOR-1206-1M -> (none)
- R106: symbol tronixio:RESISTOR-1206-36K -> tronixio:RESISTOR-1206-36K-5P; Mouser 660-RK73B2BTTD363J -> 660-RK73B2BTTDD363J; Name RESISTOR-1206-36K -> (none)
- R107: symbol tronixio:RESISTOR-1206-15K -> tronixio:RESISTOR-1206-15K-5P; Mouser 660-RK73B2BTTD153J -> 660-RK73B2BTTDD153J; Name RESISTOR-1206-15K -> (none)
- S100: footprint tronixioZZZ:E-SWITCH-200USPXT1A1M6RE -> tronixio:ZZ_E-SWITCH-200USPXT1A1M6RE
- TP100, TP101, TP102, TP103, TP104, TP105: footprint tronixioZZZ:HARWIN-S1751 -> tronixio:ZZ_HARWIN-S1751
Other:
- sheet Driver renamed Drivers
- sheet Encoder renamed Encoders
- sheet Drivers: file driver.kicad_sch -> drivers.kicad_sch
- sheet Encoders: file encoder.kicad_sch -> encoders.kicad_sch
- moved on the sheet: S100

Commit message: Up
Parts:
- added X101, X102: SYMBOL-MISC, tronixio:OSHW-5MM, symbol tronixio:OSHW-5MM
- BT100: Name KEYSTONE-1049 -> (none)
- K100: footprint tronixio:ZZ_CUI-PJ-002AH-SMT-TR -> tronixio:CUI-PJ-002AH-SMT-TR
- Q102: Name ST-STN790A-SOT-223 -> (none)
- S100: footprint tronixio:ZZ_E-SWITCH-200USPXT1A1M6RE -> tronixio:E-SWITCH-200USPXT1A1M6RE; Name E-SWITCH-200USP1T1A1M6RE -> (none)
- TH100: Name THERMISTOR-NTC-10K -> (none)
- TP100, TP101, TP102, TP103, TP104, TP105: footprint tronixio:ZZ_HARWIN-S1751 -> tronixio:HARWIN-S1751; Name HARWIN-S1751 -> (none)
- U100: Name TI-BQ2057W-SOIC -> (none)
Other:
- title: Motors Power -> Root & Motors Power
