File: Kicad/motors/drivers.kicad_sch (KiCad schematic)
At the start: 60 parts, among them K201 MOTOR 1, K202 MOTOR 2, K203 MOTOR 4, K204 MOTOR 3, U201 L298P, U202 SN74LVC1G19, U203 SN74LVC1G19, U204 L298P, U205 SN74LVC1G19, U206 SN74LVC1G19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

Commit message: Up
Parts:
- C201, C202, C205, C206, C209, C210: symbol tronixio:CAPACITOR-1206-100N -> tronixio:CAPACITOR-1206-100N-10P-X7R; Mouser 80-C1206C104M5R -> 80-C1206C104K5R; Name CAPACITOR-1206-100N -> (none); Tolerance 20% -> 10%
- C203, C204, C207, C208: footprint tronixioZZZ:CAPACITOR-ELECTROLYTIC-RADIAL-100-160-050 -> tronixio:CAPACITOR-ELECTROLYTIC-RADIAL-100-160-050; Name NICHICON-UVZ-470U-35V -> (none)
- C211, C212: symbol tronixio:CAPACITOR-1206-1U -> tronixio:CAPACITOR-1206-1U-10P-X7R; Mouser C1206C105M5RACTU -> 80-C1206C105K5R; Name CAPACITOR-1206-1U -> (none); Tolerance 20% -> 10%
- D201, D202, D203, D204, D205, D206, D207, D208, D209, D210, D211, D212, D213, D214, D215, D216: Name NEXPERIA-PMEG3030 -> (none)
- K201, K202, K203, K204: Name CUI-TB006-508-02BE -> (none)
- LED201, LED202, LED203, LED204, LED205, LED206, LED207, LED208, LED209: Name KINGBRIGHT-LED-1206-RED -> (none)
- R201, R202, R203, R206, R207, R208: symbol tronixio:RESISTOR-1206-10K -> tronixio:RESISTOR-1206-10K-5P; Name RESISTOR-1206-10K -> (none)
- R204, R205, R209, R210: symbol tronixio:RESISTOR-1210-0R5 -> tronixio:RESISTOR-1210-0R5-1P; Name RESISTOR-1210-0R5 -> (none)
- R211: symbol tronixio:RESISTOR-1206-12K -> tronixio:RESISTOR-1206-12K-5P; Mouser 660-RK73B2BTTD123J -> 660-RK73B2BTTDD103J; Name RESISTOR-1206-12K -> (none)
- TP201: footprint tronixioZZZ:HARWIN-S1751 -> tronixio:ZZ_HARWIN-S1751
- U201, U204: footprint tronixioZZZ:SOPOWER-20 -> tronixio:SOPOWER-20

Commit message: Up
Parts:
- C203, C204, C207, C208: footprint tronixio:CAPACITOR-ELECTROLYTIC-RADIAL-100-160-050 -> tronixio:ZZ_CAPACITOR-ELECTROLYTIC-RADIAL-100-160-050
Changed lines of the file:
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@@
       (effects (font (size 1.15 1.15)) (justify left))
     )
-    (property "Footprint" "tronixio:CAPACITOR-ELECTROLYTIC-RADIAL-100-160-050" (at 160.02 160.02 0)
+    (property "Footprint" "tronixio:ZZ_CAPACITOR-ELECTROLYTIC-RADIAL-100-160-050" (at 160.02 160.02 0)
       (effects (font (size 1 1)) hide)
     )
@@
       (effects (font (size 1.15 1.15)) (justify left))
     )
-    (property "Footprint" "tronixio:CAPACITOR-ELECTROLYTIC-RADIAL-100-160-050" (at 167.64 88.9 0)
+    (property "Footprint" "tronixio:ZZ_CAPACITOR-ELECTROLYTIC-RADIAL-100-160-050" (at 167.64 88.9 0)
       (effects (font (size 1 1)) hide)
     )
@@
       (effects (font (size 1.15 1.15)) (justify left))
     )
-    (property "Footprint" "tronixio:CAPACITOR-ELECTROLYTIC-RADIAL-100-160-050" (at 167.64 160.02 0)
+    (property "Footprint" "tronixio:ZZ_CAPACITOR-ELECTROLYTIC-RADIAL-100-160-050" (at 167.64 160.02 0)
       (effects (font (size 1 1)) hide)
     )
@@
       (effects (font (size 1.15 1.15)) (justify left))
     )
-    (property "Footprint" "tronixio:CAPACITOR-ELECTROLYTIC-RADIAL-100-160-050" (at 160.02 88.9 0)
-      (effects (font (size 1 1)) hide)
-    )
+    (property "Footprint" "tronixio:ZZ_CAPACITOR-ELECTROLYTIC-RADIAL-100-160-050" (at 160.02 88.9 0)
+      (effects (font (size 1 1)) hide)
+    )

Commit message: Up
Parts:
- C203, C204, C207, C208: footprint tronixio:ZZ_CAPACITOR-ELECTROLYTIC-RADIAL-100-160-050 -> tronixio:CAPACITOR-ELECTROLYTIC-RADIAL-100-160-050
- TP201: footprint tronixio:ZZ_HARWIN-S1751 -> tronixio:HARWIN-S1751; Name HARWIN-S1751 -> (none)
- U201, U204: Name ST-L298P-SOPOWER -> (none)
- U202, U203, U205, U206: Name TI-SN74LVC1G19-SOT -> (none)
- U207: Name TI-LM3480-50-SOT-23 -> (none)

Commit message: Up
Parts:
- C203, C204, C207, C208: footprint tronixio:CAPACITOR-ELECTROLYTIC-RADIAL-100-160-050 -> tronixio:CAPACITOR-ELECTROLYTIC-RADIAL-100-160-050-WURTH; symbol tronixio:NICHICON-UVZ-470U-35V -> tronixio:WURTH-WCAP-ATG8-470U-35V; Life (none) -> 2000H; Mouser UVZ1V471MPD -> 710-860010575013
- C211, C212: Mouser 80-C1206C105K5R -> 80-C1206C105K4R; Voltage 50V -> 16V

Commit message: Up
Parts:
- C201, C202, C205, C206, C209, C210: symbol tronixio:CAPACITOR-1206-100N-10P-X7R -> tronixio:CAPACITOR-1206-100N-50V-5P-X7R; Mouser 80-C1206C104K5R -> 80-C1206C104J5R; Tolerance 10% -> 5%
- C211, C212: symbol tronixio:CAPACITOR-1206-1U-10P-X7R -> tronixio:CAPACITOR-1206-1U-16V-10P-X7R
- LED201, LED202, LED203, LED204, LED205, LED206, LED207, LED208: value KINGBRIGHT-LED-1206-ORANGE -> RED
- R201, R202, R203, R206, R207, R208: value 10K -> 10k
- R211: value 12K -> 12k; Mouser 660-RK73B2BTTDD103J -> 660-RK73B2BTTD123J
- U207: symbol tronixio:TI-LM3480-50-SOT-23 -> tronixio:TI-LM3480-50-SOT
Connections:
- net VIN renamed +VIN
Other:
- moved on the sheet: C202, C203, C204, C206, C207, C208, D201, D202, D203, D204, D205, D206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

Commit message: Up
Parts:
- C203, C204, C207, C208: value 470µ/35V -> 470µ; Serie (none) -> WCAP-ATG8
- K203: value MOTOR 4 -> MOTOR 3
- K204: value MOTOR 3 -> MOTOR 4
- U202, U203, U205, U206: value SN74LVC1G19 -> 74LVC1G19; Mouser 595-SN74LVC1G19DBVR -> 595-SN74LVC1G19D
Other:
- moved on the sheet: D201, D202, D203, D204, D205, D206, D207, D208, D209, D210, D211, D212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

Commit message: Update
Parts:
- C203, C204, C207, C208: Life 2000H -> (none); Serie WCAP-ATG8 -> (none)
- D201, D202, D203, D204, D205, D206, D207, D208, D209, D210, D211, D212, D213, D214, D215, D216: symbol tronixio:NEXPERIA-PMEG3030 -> tronixio:NEXPERIA-PMEG3030-SOD
Changed lines of the file:
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@@
     (effects (font (size 1.27 1.27)) (justify right))
   )
-  (symbol (lib_id "tronixio:NEXPERIA-PMEG3030") (at 208.28 144.78 270) (unit 1)
+  (symbol (lib_id "tronixio:NEXPERIA-PMEG3030-SOD") (at 208.28 144.78 270) (unit 1)
     (in_bom yes) (on_board yes) (dnp no)
     (property "Reference" "D214" (at 209.55 147.32 0) (do_not_autoplace)
@@
     )
   )
-  (symbol (lib_id "tronixio:NEXPERIA-PMEG3030") (at 208.28 104.14 270) (unit 1)
+  (symbol (lib_id "tronixio:NEXPERIA-PMEG3030-SOD") (at 208.28 104.14 270) (unit 1)
     (in_bom yes) (on_board yes) (dnp no)
     (property "Reference" "D210" (at 209.55 101.6 0) (do_not_autoplace)
@@
       (effects (font (size 1.15 1.15)) (justify left))
     )
-    (property "Life" "2000H" (at 163.83 157.48 0)
-      (effects (font (size 1.27 1.27)) (justify left) hide)
-    )
-    (property "Serie" "WCAP-ATG8" (at 162.56 167.64 0)
-      (effects (font (size 1 1)) hide)
-    )
     (pin "1")
     (pin "2")
@@
     )
   )
-  (symbol (lib_id "tronixio:NEXPERIA-PMEG3030") (at 208.28 33.02 270) (unit 1)
+  (symbol (lib_id "tronixio:NEXPERIA-PMEG3030-SOD") (at 208.28 33.02 270) (unit 1)
     (in_bom yes) (on_board yes) (dnp no)
     (property "Reference" "D202" (at 209.55 31.115 0) (do_not_autoplace)
@@
       (effects (font (size 1.15 1.15)) (justify left))
     )
-    (property "Life" "2000H" (at 171.45 86.36 0)
-      (effects (font (size 1.27 1.27)) (justify left) hide)
-    )
-    (property "Serie" "WCAP-ATG8" (at 170.18 96.52 0)
-      (effects (font (size 1 1)) hide)
-    )
     (pin "1")
     (pin "2")
@@
     )
   )
-  (symbol (lib_id "tronixio:NEXPERIA-PMEG3030") (at 215.9 144.78 270) (unit 1)
+  (symbol (lib_id "tronixio:NEXPERIA-PMEG3030-SOD") (at 215.9 144.78 270) (unit 1)
     (in_bom yes) (on_board yes) (dnp no)
     (property "Reference" "D215" (at 217.17 147.32 0) (do_not_autoplace)
@@
     )
   )
-  (symbol (lib_id "tronixio:NEXPERIA-PMEG3030") (at 215.9 104.14 270) (unit 1)
+  (symbol (lib_id "tronixio:NEXPERIA-PMEG3030-SOD") (at 215.9 104.14 270) (unit 1)
     (in_bom yes) (on_board yes) (dnp no)
     (property "Reference" "D211" (at 217.17 101.6 0) (do_not_autoplace)
@@
     )
   )
-  (symbol (lib_id "tronixio:NEXPERIA-PMEG3030") (at 200.66 104.14 270) (unit 1)
+  (symbol (lib_id "tronixio:NEXPERIA-PMEG3030-SOD") (at 200.66 104.14 270) (unit 1)
     (in_bom yes) (on_board yes) (dnp no)
     (property "Reference" "D209" (at 201.93 101.6 0) (do_not_autoplace)
@@
     )
   )
-  (symbol (lib_id "tronixio:NEXPERIA-PMEG3030") (at 223.52 33.02 270) (unit 1)
+  (symbol (lib_id "tronixio:NEXPERIA-PMEG3030-SOD") (at 223.52 33.02 270) (unit 1)
     (in_bom yes) (on_board yes) (dnp no)
     (property "Reference" "D204" (at 224.79 31.115 0) (do_not_autoplace)
@@
     )
   )
-  (symbol (lib_id "tronixio:NEXPERIA-PMEG3030") (at 200.66 33.02 270) (unit 1)
+  (symbol (lib_id "tronixio:NEXPERIA-PMEG3030-SOD") (at 200.66 33.02 270) (unit 1)
     (in_bom yes) (on_board yes) (dnp no)
     (property "Reference" "D201" (at 201.93 31.115 0) (do_not_autoplace)
@@
     )
   )
-  (symbol (lib_id "tronixio:NEXPERIA-PMEG3030") (at 223.52 144.78 270) (unit 1)
+  (symbol (lib_id "tronixio:NEXPERIA-PMEG3030-SOD") (at 223.52 144.78 270) (unit 1)
     (in_bom yes) (on_board yes) (dnp no)
     (property "Reference" "D216" (at 224.79 147.32 0) (do_not_autoplace)
@@
     )
   )
-  (symbol (lib_id "tronixio:NEXPERIA-PMEG3030") (at 215.9 73.66 270) (unit 1)
+  (symbol (lib_id "tronixio:NEXPERIA-PMEG3030-SOD") (at 215.9 73.66 270) (unit 1)
     (in_bom yes) (on_board yes) (dnp no)
     (property "Reference" "D207" (at 217.17 76.2 0) (do_not_autoplace)
@@
     )
   )
-  (symbol (lib_id "tronixio:NEXPERIA-PMEG3030") (at 223.52 73.66 270) (unit 1)
+  (symbol (lib_id "tronixio:NEXPERIA-PMEG3030-SOD") (at 223.52 73.66 270) (unit 1)
     (in_bom yes) (on_board yes) (dnp no)
     (property "Reference" "D208" (at 224.79 76.2 0) (do_not_autoplace)
@@
     )
   )
-  (symbol (lib_id "tronixio:NEXPERIA-PMEG3030") (at 208.28 73.66 270) (unit 1)
+  (symbol (lib_id "tronixio:NEXPERIA-PMEG3030-SOD") (at 208.28 73.66 270) (unit 1)
     (in_bom yes) (on_board yes) (dnp no)
     (property "Reference" "D206" (at 209.55 76.2 0) (do_not_autoplace)
@@
     (property "Voltage" "35V" (at 170.815 154.94 0) (do_not_autoplace)
       (effects (font (size 1.15 1.15)) (justify left))
-    )
-    (property "Life" "2000H" (at 171.45 157.48 0)
-      (effects (font (size 1.27 1.27)) (justify left) hide)
-    )
-    (property "Serie" "WCAP-ATG8" (at 170.18 167.64 0)
-      (effects (font (size 1 1)) hide)
     )
     (pin "1")
@@
     )
   )
-  (symbol (lib_id "tronixio:NEXPERIA-PMEG3030") (at 200.66 144.78 270) (unit 1)
+  (symbol (lib_id "tronixio:NEXPERIA-PMEG3030-SOD") (at 200.66 144.78 270) (unit 1)
     (in_bom yes) (on_board yes) (dnp no)
     (property "Reference" "D213" (at 201.93 147.32 0) (do_not_autoplace)
@@
     )
   )
-  (symbol (lib_id "tronixio:NEXPERIA-PMEG3030") (at 200.66 73.66 270) (unit 1)
+  (symbol (lib_id "tronixio:NEXPERIA-PMEG3030-SOD") (at 200.66 73.66 270) (unit 1)
     (in_bom yes) (on_board yes) (dnp no)
     (property "Reference" "D205" (at 201.93 76.2 0) (do_not_autoplace)
@@
     )
   )
-  (symbol (lib_id "tronixio:NEXPERIA-PMEG3030") (at 215.9 33.02 270) (unit 1)
+  (symbol (lib_id "tronixio:NEXPERIA-PMEG3030-SOD") (at 215.9 33.02 270) (unit 1)
     (in_bom yes) (on_board yes) (dnp no)
     (property "Reference" "D203" (at 217.17 31.115 0) (do_not_autoplace)
@@
       (effects (font (size 1.15 1.15)) (justify left))
     )
-    (property "Life" "2000H" (at 163.83 86.36 0)
-      (effects (font (size 1.27 1.27)) (justify left) hide)
-    )
-    (property "Serie" "WCAP-ATG8" (at 162.56 96.52 0)
-      (effects (font (size 1 1)) hide)
-    )
     (pin "1")
     (pin "2")
@@
     )
   )
-  (symbol (lib_id "tronixio:NEXPERIA-PMEG3030") (at 223.52 104.14 270) (unit 1)
+  (symbol (lib_id "tronixio:NEXPERIA-PMEG3030-SOD") (at 223.52 104.14 270) (unit 1)
     (in_bom yes) (on_board yes) (dnp no)
     (property "Reference" "D212" (at 224.79 101.6 0) (do_not_autoplace)
