File: Kicad/motors/encoders.kicad_sch (KiCad schematic)
At the start: 28 parts, among them K301 FRONT, K302 REAR, Q301 BC846BS, Q302 BC846BS, U301 SN74LVC2G17, U302 SN74LVC2G17, U303 LM3480-33

Commit message: Up
Parts:
- C301, C303: symbol tronixio:CAPACITOR-1206-100N -> tronixio:CAPACITOR-1206-100N-10P-X7R; Mouser 80-C1206C104M5R -> 80-C1206C104K5R; Name CAPACITOR-1206-100N -> (none); Tolerance 20% -> 10%
- C302, C304, C305, C306: symbol tronixio:CAPACITOR-1206-1U -> tronixio:CAPACITOR-1206-1U-10P-X7R; Mouser C1206C105M5RACTU -> 80-C1206C105K5R; Name CAPACITOR-1206-1U -> (none); Tolerance 20% -> 10%
- IR301, IR302, IR303, IR304: footprint tronixioZZZ:OPB-610 -> tronixio:ZZ_OPB-610
- K301, K302: Name HARWIN-254-F-1X10-VERTICAL -> (none)
- LED301: Name KINGBRIGHT-LED-1206-RED -> (none)
- Q301, Q302: footprint tronixioZZZ:SOT-70-6 -> tronixio:SC-70-6
- R301, R302, R303, R304: symbol tronixio:RESISTOR-1206-10K -> tronixio:RESISTOR-1206-10K-5P; Name RESISTOR-1206-10K -> (none)
- R305, R306: symbol tronixio:RESISTOR-1206-2K2 -> tronixio:RESISTOR-1206-2K2-5P; Mouser 660-RK73B2BTTD222J -> 660-RK73B2BTTDD222J; Name RESISTOR-1206-2K2 -> (none)
- R307, R308: symbol tronixio:RESISTOR-1206-33R -> tronixio:RESISTOR-1206-33R-5P; Name RESISTOR-1206-33R -> (none)
- R309: symbol tronixio:RESISTOR-1206-6K8 -> tronixio:RESISTOR-1206-6K8-5P; Name RESISTOR-1206-6K8 -> (none)
- TP301: footprint tronixioZZZ:HARWIN-S1751 -> tronixio:ZZ_HARWIN-S1751

Commit message: Up
Parts:
- IR301, IR302, IR303, IR304: footprint tronixio:ZZ_OPB-610 -> tronixio:OPB-610; Name TTE-OPB610 -> (none)
- Q301, Q302: Name NEXPERIA-BC846BS -> (none)
- TP301: footprint tronixio:ZZ_HARWIN-S1751 -> tronixio:HARWIN-S1751; Name HARWIN-S1751 -> (none)
- U301, U302: Name TI-SN74LVC2G17-SOT -> (none)
- U303: Name TI-LM3480-33-SOT-23 -> (none)

Commit message: Up
Parts:
- C302, C304, C305, C306: Mouser 80-C1206C105K5R -> 80-C1206C105K4R; Voltage 50V -> 16V
Changed lines of the file:
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@@
       (effects (font (size 1 1)) hide)
     )
-    (property "Voltage" "50V" (at 114.22 182.88 0) (do_not_autoplace)
+    (property "Voltage" "16V" (at 114.22 182.88 0) (do_not_autoplace)
       (effects (font (size 1.15 1.15)) (justify left) hide)
     )
@@
       (effects (font (size 1.15 1.15)) (justify left) hide)
     )
-    (property "Mouser" "80-C1206C105K5R" (at 109.22 190.5 0)
+    (property "Mouser" "80-C1206C105K4R" (at 109.22 190.5 0)
       (effects (font (size 1 1)) hide)
     )
@@
       (effects (font (size 1 1)) hide)
     )
-    (property "Voltage" "50V" (at 50.72 185.42 0) (do_not_autoplace)
+    (property "Voltage" "16V" (at 50.72 185.42 0) (do_not_autoplace)
       (effects (font (size 1.15 1.15)) (justify left) hide)
     )
@@
       (effects (font (size 1.15 1.15)) (justify left) hide)
     )
-    (property "Mouser" "80-C1206C105K5R" (at 45.72 193.04 0)
+    (property "Mouser" "80-C1206C105K4R" (at 45.72 193.04 0)
       (effects (font (size 1 1)) hide)
     )
@@
       (effects (font (size 1 1)) hide)
     )
-    (property "Voltage" "50V" (at 30.4 185.42 0) (do_not_autoplace)
+    (property "Voltage" "16V" (at 30.4 185.42 0) (do_not_autoplace)
       (effects (font (size 1.15 1.15)) (justify left) hide)
     )
@@
       (effects (font (size 1.15 1.15)) (justify left) hide)
     )
-    (property "Mouser" "80-C1206C105K5R" (at 25.4 193.04 0)
+    (property "Mouser" "80-C1206C105K4R" (at 25.4 193.04 0)
       (effects (font (size 1 1)) hide)
     )
@@
       (effects (font (size 1 1)) hide)
     )
-    (property "Voltage" "50V" (at 137.08 182.88 0) (do_not_autoplace)
+    (property "Voltage" "16V" (at 137.08 182.88 0) (do_not_autoplace)
       (effects (font (size 1.15 1.15)) (justify left) hide)
     )
@@
       (effects (font (size 1.15 1.15)) (justify left) hide)
     )
-    (property "Mouser" "80-C1206C105K5R" (at 132.08 190.5 0)
-      (effects (font (size 1 1)) hide)
-    )
+    (property "Mouser" "80-C1206C105K4R" (at 132.08 190.5 0)
+      (effects (font (size 1 1)) hide)
+    )

Commit message: Up
Parts:
- C301, C303: symbol tronixio:CAPACITOR-1206-100N-10P-X7R -> tronixio:CAPACITOR-1206-100N-50V-5P-X7R; Mouser 80-C1206C104K5R -> 80-C1206C104J5R; Tolerance 10% -> 5%
- C302, C304, C305, C306: symbol tronixio:CAPACITOR-1206-1U-10P-X7R -> tronixio:CAPACITOR-1206-1U-16V-10P-X7R
- R301, R302, R303, R304: value 10K -> 10k
- R305, R306: value 2K2 -> 2k2
- R309: value 6K8 -> 6k8; Mouser 660-RK73B2BTTDD682J -> 660-RK73B2BTTD682J
- U303: symbol tronixio:TI-LM3480-33-SOT-23 -> tronixio:TI-LM3480-33-SOT
Connections:
- net VIN renamed +VIN

Commit message: Up
Parts:
- Q301, Q302: symbol tronixio:NEXPERIA-BC846BS -> tronixio:NEXPERIA-BC846BS-SC
- U301, U302: value SN74LVC2G17 -> 74LVC2G17; Mouser 595-SN74LVC2G17DBVR -> 595-SN74LVC2G17D

Commit message: Update
Changed lines of the file:
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@@
       (effects (font (size 1 1)) hide)
     )
-    (property "Datasheet" "https://www.ttelectronics.com/products/categories/optoelectronics/optoelectronics/opb610/" (at 195.58 106.68 0) (do_not_autoplace)
+    (property "Datasheet" "https://www.ttelectronics.com/Products/Sensors/Optoelectronics/Slotted-Switches/OPB610" (at 195.58 106.68 0) (do_not_autoplace)
       (effects (font (size 1 1)) hide)
     )
@@
       (effects (font (size 1 1)) hide)
     )
-    (property "Datasheet" "https://www.ttelectronics.com/products/categories/optoelectronics/optoelectronics/opb610/" (at 93.98 68.58 0) (do_not_autoplace)
+    (property "Datasheet" "https://www.ttelectronics.com/Products/Sensors/Optoelectronics/Slotted-Switches/OPB610" (at 93.98 68.58 0) (do_not_autoplace)
       (effects (font (size 1 1)) hide)
     )
@@
       (effects (font (size 1 1)) hide)
     )
-    (property "Datasheet" "https://www.ttelectronics.com/products/categories/optoelectronics/optoelectronics/opb610/" (at 93.98 106.68 0) (do_not_autoplace)
+    (property "Datasheet" "https://www.ttelectronics.com/Products/Sensors/Optoelectronics/Slotted-Switches/OPB610" (at 93.98 106.68 0) (do_not_autoplace)
       (effects (font (size 1 1)) hide)
     )
@@
       (effects (font (size 1 1)) hide)
     )
-    (property "Datasheet" "https://www.ttelectronics.com/products/categories/optoelectronics/optoelectronics/opb610/" (at 195.58 68.58 0) (do_not_autoplace)
-      (effects (font (size 1 1)) hide)
-    )
+    (property "Datasheet" "https://www.ttelectronics.com/Products/Sensors/Optoelectronics/Slotted-Switches/OPB610" (at 195.58 68.58 0) (do_not_autoplace)
+      (effects (font (size 1 1)) hide)
+    )
