File: Kicad/motors/main.kicad_sch (KiCad schematic)
At the start: 49 parts, among them K100 9V - 1A, Q100 DMP2305U, Q101 DMP2305U, Q102 STN790A, U100 BQ2057W, X101 SYMBOL-MISC, X102 SYMBOL-MISC

Commit message: Up
Parts:
- C101: Mouser 80-C1206C105K5R -> 80-C1206C105K4R; Voltage 50V -> 16V
- R100, R101: Tolerance 5% -> 1%
Changed lines of the file:
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@@
       (effects (font (size 1 1)) hide)
     )
-    (property "Tolerance" "5%" (at 199.39 38.1 0) (do_not_autoplace)
-      (effects (font (size 1.15 1.15)) (justify left) hide)
+    (property "Tolerance" "1%" (at 198.755 39.37 90) (do_not_autoplace)
+      (effects (font (size 1.15 1.15)) (justify right))
     )
     (property "Mouser" "660-SR732ETTER100F" (at 210.82 40.64 0)
@@
       (effects (font (size 1 1)) hide)
     )
-    (property "Voltage" "50V" (at 225.98 81.28 0) (do_not_autoplace)
+    (property "Voltage" "16V" (at 225.98 81.28 0) (do_not_autoplace)
       (effects (font (size 1.15 1.15)) (justify left) hide)
     )
@@
       (effects (font (size 1.15 1.15)) (justify left) hide)
     )
-    (property "Mouser" "80-C1206C105K5R" (at 220.98 88.9 0)
+    (property "Mouser" "80-C1206C105K4R" (at 220.98 88.9 0)
       (effects (font (size 1 1)) hide)
     )
@@
       (effects (font (size 1 1)) hide)
     )
-    (property "Tolerance" "5%" (at 199.39 43.18 0) (do_not_autoplace)
-      (effects (font (size 1.15 1.15)) (justify left) hide)
+    (property "Tolerance" "1%" (at 198.755 44.45 90) (do_not_autoplace)
+      (effects (font (size 1.15 1.15)) (justify right))
     )
     (property "Mouser" "660-SR732ETTER100F" (at 210.82 45.72 0)

Commit message: Up
Parts:
- C100: symbol tronixio:CAPACITOR-1206-100N-10P-X7R -> tronixio:CAPACITOR-1206-100N-50V-5P-X7R; Mouser 80-C1206C104K5R -> 80-C1206C104J5R; Tolerance 10% -> 5%
- C101: symbol tronixio:CAPACITOR-1206-1U-10P-X7R -> tronixio:CAPACITOR-1206-1U-16V-10P-X7R
- LED100: value CHARGE -> Charge
- LED101: value POWER -> RED
- Q100, Q101: symbol tronixio:DIODES-DMP2305U-SOT-23 -> tronixio:DIODES-DMP2305U-SOT
- R100, R101: footprint tronixio:RESISTOR-SMD-1206 -> tronixio:RESISTOR-SMD-1210; symbol tronixio:RESISTOR-1206-0R1-5P -> tronixio:RESISTOR-1210-0R1-1P
- R102: value 1K -> 1k
- R103, R105: value 10K -> 10k
- R106: value 36K -> 36k
- R107: value 15K -> 15k
- TH100: value NTC-10K -> 10k
- TP104, TP105: value KEYSTONE-2000-3 -> HARWIN-S1751
- U100: symbol tronixio:TI-BQ2057W-SOIC-08 -> tronixio:TI-BQ2057W-SOIC
- X101, X102: value SYMBOL-MISC -> OSHW-5MM
Connections:
- net VBAT renamed +VBAT
- net VCC renamed +VCC
- net VIN renamed +VIN

Commit message: Up
Parts:
- K100: value 9V - 1A -> PJ-102H
- LED101: value RED -> Power
Changed lines of the file:
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@@
     (effects (font (size 4 4)) (justify left bottom))
   )
-  (text "*R101: Optional, needed for adjust precise value." (at 180.34 171.45 0)
+  (text "*R101: Optional, needed for adjust precise value." (at 180.975 171.45 0)
     (effects (font (size 1.27 1.27)) (justify left bottom))
   )
@@
     (effects (font (size 1.27 1.27)) (justify right bottom))
   )
-  (text "*R106: 10K if NTC TH100 Not Populate." (at 180.34 173.99 0)
+  (text "*R106: 10K if NTC TH100 Not Populate." (at 180.975 173.99 0)
     (effects (font (size 1.27 1.27)) (justify left bottom))
   )
-  (text "R100 (0Ω1): ICharge ~1A." (at 180.34 168.91 0)
+  (text "R100 (0Ω1): ICharge ~1A." (at 180.975 168.91 0)
     (effects (font (size 1.27 1.27)) (justify left bottom))
   )
@@
     )
   )
-  (symbol (lib_name "POWER-GND_10") (lib_id "tronixio:POWER-GND") (at 177.8 83.82 0) (unit 1)
+  (symbol (lib_id "tronixio:POWER-GND") (at 177.8 83.82 0) (unit 1)
     (in_bom yes) (on_board yes) (dnp no)
     (property "Reference" "#PWR0102" (at 177.8 88.9 0)
@@
     )
   )
-  (symbol (lib_name "POWER-GND_11") (lib_id "tronixio:POWER-GND") (at 68.58 83.82 0) (unit 1)
+  (symbol (lib_id "tronixio:POWER-GND") (at 68.58 83.82 0) (unit 1)
     (in_bom yes) (on_board yes) (dnp no)
     (property "Reference" "#PWR0119" (at 68.58 88.9 0)
@@
   (symbol (lib_id "tronixio:E-SWITCH-200USP1T1A1M6RE") (at 86.36 76.2 90) (unit 1)
     (in_bom yes) (on_board yes) (dnp no)
-    (property "Reference" "S100" (at 86.36 71.12 90) (do_not_autoplace)
+    (property "Reference" "S100" (at 86.36 83.185 90) (do_not_autoplace)
       (effects (font (size 1.15 1.15)) (justify left))
     )
@@
     )
   )
-  (symbol (lib_name "POWER-GND_16") (lib_id "tronixio:POWER-GND") (at 50.8 124.46 0) (unit 1)
+  (symbol (lib_id "tronixio:POWER-GND") (at 50.8 124.46 0) (unit 1)
     (in_bom yes) (on_board yes) (dnp no)
     (property "Reference" "#PWR0120" (at 50.8 129.54 0)
@@
   (symbol (lib_id "tronixio:ST-STN790A-SOT-223") (at 213.36 43.18 270) (mirror x) (unit 1)
     (in_bom yes) (on_board yes) (dnp no)
-    (property "Reference" "Q102" (at 213.36 34.29 90)
+    (property "Reference" "Q102" (at 213.36 34.29 90) (do_not_autoplace)
       (effects (font (size 1.15 1.15)))
     )
@@
       (effects (font (size 1 1)) hide)
     )
-    (property "Tolerance" "1%" (at 198.755 41.91 90) (do_not_autoplace)
+    (property "Tolerance" "1%" (at 198.755 39.37 90) (do_not_autoplace)
       (effects (font (size 1.15 1.15)) (justify right))
     )
@@
   (symbol (lib_id "tronixio:KEYSTONE-1049") (at 50.8 76.2 0) (unit 2)
     (in_bom yes) (on_board yes) (dnp no)
-    (property "Reference" "BT100" (at 49.53 78.74 0)
+    (property "Reference" "BT100" (at 49.53 78.74 0) (do_not_autoplace)
       (effects (font (size 1.15 1.15)) (justify right))
     )
@@
     )
   )
-  (symbol (lib_name "POWER-GND_2") (lib_id "tronixio:POWER-GND") (at 93.98 124.46 0) (unit 1)
+  (symbol (lib_id "tronixio:POWER-GND") (at 93.98 124.46 0) (unit 1)
     (in_bom yes) (on_board yes) (dnp no)
     (property "Reference" "#PWR0114" (at 93.98 129.54 0)
@@
   (symbol (lib_id "tronixio:KINGBRIGHT-LED-1206-RED") (at 50.8 119.38 90) (unit 1)
     (in_bom yes) (on_board yes) (dnp no)
-    (property "Reference" "LED101" (at 50.165 115.57 90)
+    (property "Reference" "LED101" (at 50.165 115.57 90) (do_not_autoplace)
       (effects (font (size 1.15 1.15)) (justify left))
     )
-    (property "Value" "RED" (at 50.165 121.92 0) (do_not_autoplace)
-      (effects (font (size 1.15 1.15)))
+    (property "Value" "Power" (at 50.165 121.92 90) (do_not_autoplace)
+      (effects (font (size 1.15 1.15)) (justify left))
     )
     (property "Footprint" "tronixio:LED-SMD-1206" (at 58.42 119.38 0) (do_not_autoplace)
@@
   (symbol (lib_id "tronixio:KEYSTONE-1049") (at 50.8 68.58 0) (unit 1)
     (in_bom yes) (on_board yes) (dnp no)
-    (property "Reference" "BT100" (at 49.53 63.5 0)
+    (property "Reference" "BT100" (at 49.53 63.5 0) (do_not_autoplace)
       (effects (font (size 1.15 1.15)) (justify right))
     )
@@
     )
   )
-  (symbol (lib_name "POWER-GND_3") (lib_id "tronixio:POWER-GND") (at 160.02 83.82 0) (unit 1)
+  (symbol (lib_id "tronixio:POWER-GND") (at 160.02 83.82 0) (unit 1)
     (in_bom yes) (on_board yes) (dnp no)
     (property "Reference" "#PWR0111" (at 160.02 88.9 0)
@@
     )
   )
-  (symbol (lib_name "POWER-GND_4") (lib_id "tronixio:POWER-GND") (at 228.6 83.82 0) (unit 1)
+  (symbol (lib_id "tronixio:POWER-GND") (at 228.6 83.82 0) (unit 1)
     (in_bom yes) (on_board yes) (dnp no)
     (property "Reference" "#PWR0123" (at 228.6 88.9 0)
@@
   (symbol (lib_id "tronixio:CAPACITOR-1206-1U-16V-10P-X7R") (at 220.98 76.2 0) (unit 1)
     (in_bom yes) (on_board yes) (dnp no)
-    (property "Reference" "C101" (at 221.615 73.66 0)
+    (property "Reference" "C101" (at 221.615 73.66 0) (do_not_autoplace)
       (effects (font (size 1.15 1.15)) (justify left))
     )
@@
     )
   )
-  (symbol (lib_name "POWER-GND_1") (lib_id "tronixio:POWER-GND") (at 175.26 190.5 0) (unit 1)
+  (symbol (lib_id "tronixio:POWER-GND") (at 175.26 190.5 0) (unit 1)
     (in_bom yes) (on_board yes) (dnp no)
     (property "Reference" "#PWR0108" (at 175.26 195.58 0)
@@
     (property "Datasheet" "" (at 175.26 190.5 0)
       (effects (font (size 1 1)) hide)
-    )
-    (property "Name" "GND" (at 175.26 194.31 0)
-      (effects (font (size 1.15 1.15)) hide)
     )
     (pin "1")
@@
     )
   )
-  (symbol (lib_name "POWER-GND_5") (lib_id "tronixio:POWER-GND") (at 106.68 124.46 0) (unit 1)
+  (symbol (lib_id "tronixio:POWER-GND") (at 106.68 124.46 0) (unit 1)
     (in_bom yes) (on_board yes) (dnp no)
     (property "Reference" "#PWR0113" (at 106.68 129.54 0)
@@
     )
   )
-  (symbol (lib_name "POWER-GND_6") (lib_id "tronixio:POWER-GND") (at 220.98 83.82 0) (unit 1)
+  (symbol (lib_id "tronixio:POWER-GND") (at 220.98 83.82 0) (unit 1)
     (in_bom yes) (on_board yes) (dnp no)
     (property "Reference" "#PWR0121" (at 220.98 88.9 0)
@@
     )
   )
-  (symbol (lib_name "POWER-GND_7") (lib_id "tronixio:POWER-GND") (at 68.58 124.46 0) (unit 1)
+  (symbol (lib_id "tronixio:POWER-GND") (at 68.58 124.46 0) (unit 1)
     (in_bom yes) (on_board yes) (dnp no)
     (property "Reference" "#PWR0116" (at 68.58 129.54 0)
@@
     )
   )
-  (symbol (lib_name "POWER-GND_8") (lib_id "tronixio:POWER-GND") (at 81.28 124.46 0) (unit 1)
+  (symbol (lib_id "tronixio:POWER-GND") (at 81.28 124.46 0) (unit 1)
     (in_bom yes) (on_board yes) (dnp no)
     (property "Reference" "#PWR0115" (at 81.28 129.54 0)
@@
     )
   )
-  (symbol (lib_name "POWER-GND_9") (lib_id "tronixio:POWER-GND") (at 185.42 83.82 0) (unit 1)
+  (symbol (lib_id "tronixio:POWER-GND") (at 185.42 83.82 0) (unit 1)
     (in_bom yes) (on_board yes) (dnp no)
     (property "Reference" "#PWR0101" (at 185.42 88.9 0)
@@
     )
   )
-  (symbol (lib_name "POWER-GND_12") (lib_id "tronixio:POWER-GND") (at 88.9 83.82 0) (unit 1)
+  (symbol (lib_id "tronixio:POWER-GND") (at 88.9 83.82 0) (unit 1)
     (in_bom yes) (on_board yes) (dnp no)
     (property "Reference" "#PWR0112" (at 88.9 88.9 0)
@@
     )
   )
-  (symbol (lib_name "POWER-GND_13") (lib_id "tronixio:POWER-GND") (at 50.8 83.82 0) (unit 1)
+  (symbol (lib_id "tronixio:POWER-GND") (at 50.8 83.82 0) (unit 1)
     (in_bom yes) (on_board yes) (dnp no)
     (property "Reference" "#PWR0118" (at 50.8 88.9 0)
@@
       (effects (font (size 1 1)) hide)
     )
-    (property "Tolerance" "1%" (at 198.755 46.99 90) (do_not_autoplace)
+    (property "Tolerance" "1%" (at 198.755 44.45 90) (do_not_autoplace)
       (effects (font (size 1.15 1.15)) (justify right))
     )
@@
     )
   )
-  (symbol (lib_name "POWER-GND_14") (lib_id "tronixio:POWER-GND") (at 170.18 83.82 0) (unit 1)
+  (symbol (lib_id "tronixio:POWER-GND") (at 170.18 83.82 0) (unit 1)
     (in_bom yes) (on_board yes) (dnp no)
     (property "Reference" "#PWR0103" (at 170.18 88.9 0)
@@
       (effects (font (size 1.15 1.15)))
     )
-    (property "Value" "9V - 1A" (at 152.4 60.96 0) (do_not_autoplace)
+    (property "Value" "PJ-102H" (at 152.4 60.96 0) (do_not_autoplace)
       (effects (font (size 1.15 1.15)))
     )
@@
     )
   )
-  (symbol (lib_name "POWER-GND_15") (lib_id "tronixio:POWER-GND") (at 236.22 83.82 0) (unit 1)
+  (symbol (lib_id "tronixio:POWER-GND") (at 236.22 83.82 0) (unit 1)
     (in_bom yes) (on_board yes) (dnp no)
     (property "Reference" "#PWR0122" (at 236.22 88.9 0)
@@
   (symbol (lib_id "tronixio:TI-BQ2057W-SOIC") (at 187.96 55.88 0) (unit 1)
     (in_bom yes) (on_board yes) (dnp no)
-    (property "Reference" "U100" (at 195.58 52.07 0)
+    (property "Reference" "U100" (at 195.58 52.07 0) (do_not_autoplace)
       (effects (font (size 1.15 1.15)))
     )
@@
     (stroke (width 0.001) (type solid))
     (fill (color 0 0 0 0.0000))
-    (property "Sheetname" "Encoders" (at 88.9 146.7191 0)
+    (property "Sheetname" "Encoders" (at 88.9 146.7191 0) (do_not_autoplace)
       (effects (font (size 2 2)) (justify left bottom))
     )
-    (property "Sheetfile" "encoders.kicad_sch" (at 88.9 182.88 0)
+    (property "Sheetfile" "encoders.kicad_sch" (at 88.9 182.88 0) (do_not_autoplace)
       (effects (font (size 1.27 1.27)) (justify left top))
     )
@@
     (stroke (width 0.001) (type solid))
     (fill (color 0 0 0 0.0000))
-    (property "Sheetname" "Drivers" (at 38.1 146.6841 0)
+    (property "Sheetname" "Drivers" (at 38.1 146.6841 0) (do_not_autoplace)
       (effects (font (size 2 2)) (justify left bottom))
     )
-    (property "Sheetfile" "drivers.kicad_sch" (at 38.1 182.88 0)
+    (property "Sheetfile" "drivers.kicad_sch" (at 38.1 182.88 0) (do_not_autoplace)
       (effects (font (size 1.27 1.27)) (justify left top))
     )

Commit message: Up
Other:
- note added: "*R106: 10k if NTC TH100 Not Populate."
- note removed: "*R106: 10K if NTC TH100 Not Populate."
Changed lines of the file:
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@@
     (effects (font (size 1.27 1.27)) (justify right bottom))
   )
-  (text "*R106: 10K if NTC TH100 Not Populate." (at 180.975 173.99 0)
+  (text "*R106: 10k if NTC TH100 Not Populate." (at 180.975 173.99 0)
     (effects (font (size 1.27 1.27)) (justify left bottom))
   )
@@
   (symbol (lib_id "tronixio:E-SWITCH-200USP1T1A1M6RE") (at 86.36 76.2 90) (unit 1)
     (in_bom yes) (on_board yes) (dnp no)
-    (property "Reference" "S100" (at 86.36 83.185 90) (do_not_autoplace)
+    (property "Reference" "S100" (at 86.36 83.82 90) (do_not_autoplace)
       (effects (font (size 1.15 1.15)) (justify left))
     )

Commit message: Update
Parts:
- D100: symbol tronixio:NEXPERIA-PMEG3030 -> tronixio:NEXPERIA-PMEG3030-SOD
Changed lines of the file:
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@@
     )
   )
-  (symbol (lib_id "tronixio:NEXPERIA-PMEG3030") (at 170.18 55.88 0) (mirror y) (unit 1)
+  (symbol (lib_id "tronixio:NEXPERIA-PMEG3030-SOD") (at 170.18 55.88 0) (mirror y) (unit 1)
     (in_bom yes) (on_board yes) (dnp no)
     (property "Reference" "D100" (at 170.18 53.34 0) (do_not_autoplace)
