File: Kicad/ir/ir.kicad_pcb (KiCad board)
At the start: 2 copper layers, 150 x 35 mm, 20 parts, among them IC1 LITEON-LTH-1550-01, IC2 LITEON-LTH-1550-01, IC3 LITEON-LTH-1550-01, Q1 BC846BS

Commit message: Update
Parts:
- removed H5, H6, H7, H8: MOUNTING-HOLE-MASK-3MM, tronixio:M3-MASK
- removed IC3: LITEON-LTH-1550-01, tronixio:zzzLTH-1550-01-HORIZONTAL
- removed TP1: HARWIN-S1751, tronixio:zzzHARWIN-S1751
- added C1: C-1206, tronixio:KEMET-C322, F.Cu at (165.7, 84.8)
- added C2: C-1206, tronixio:KEMET-C322, F.Cu at (142.9, 84.8)
- added JP1: HARWIN-254-M-1X02-JUMPER-VERTICAL, tronixio:HARWIN-M20-999024x, F.Cu at (132.7, 73.3)
- added K1: HARWIN-254-M-1X04-VERTICAL, tronixio:HARWIN-M20-999044x, F.Cu at (188.6, 82.2)
- added K2: HARWIN-254-M-1X05-VERTICAL, tronixio:HARWIN-M20-999054x, F.Cu at (155.6, 96.2)
- added K3: HARWIN-254-M-1X02-VERTICAL, tronixio:HARWIN-M20-999024x, F.Cu at (179.7, 96.2)
- added K4: HARWIN-254-M-1X02-VERTICAL, tronixio:HARWIN-M20-999024x, F.Cu at (108.6, 83.5)
- added Q2: ONSEMI-BC546-TO92, tronixio:TO-92-INLINE, F.Cu at (118.8, 92.4)
- added R5: R-1206, tronixio:RESISTOR-1016-TH, F.Cu at (130.2, 84.8)
- added R6: R-1206, tronixio:RESISTOR-1016-TH, F.Cu at (161.9, 84.8)
- added R7: R-1206, tronixio:RESISTOR-1016-TH, F.Cu at (135.3, 84.8)
- added R8: R-1206, tronixio:RESISTOR-1016-TH, F.Cu at (125.1, 84.8)
- added R9: R-1206, tronixio:RESISTOR-1016-TH, F.Cu at (174.6, 84.8)
- added U1: MICROCHIP-MCP6541-DIP-08, tronixio:DIP-08-W762, F.Cu at (146.7, 88.6)
- IC2: footprint tronixio:zzzLTH-1550-01-HORIZONTAL -> tronixio:zzzLTH-1550-01-VERTICAL; moved to F.Cu
- LED1: value Power -> LED-1206-RED; footprint tronixio:LED-1206 -> tronixio:LED-05MM-TH; moved to F.Cu
- Q1: value BC846BS -> ONSEMI-BC546-TO92; footprint tronixio:SOT-23-6 -> tronixio:TO-92-INLINE
- R1: value 4K7 -> R-1206
- R2: value 2K7 -> R-1206
- R3: value 33Ω -> R-1206
- R4: value 6K8 -> R-1206; footprint tronixio:RESISTOR-1206 -> tronixio:RESISTOR-1016-TH
- moved R1 130.4 mm to (169.6, 84.8), turned to -90 degrees
- moved H4 123.6 mm to (201.5, 86.5)
- moved H3 115.7 mm to (181.5, 78.0)
- moved R3 113.4 mm to (158.1, 84.8), turned to -90 degrees
- moved IC1 104.6 mm to (150.5, 69.0), turned to 0 degrees
- moved G*** 91.5 mm to (99.7, 96.2)
- moved G*** 91.1 mm to (83.7, 96.2)
- moved LED1 89.3 mm to (181.0, 87.3), turned to -90 degrees
- moved R2 88.4 mm to (139.1, 84.8), turned to 90 degrees
- moved IC2 78.9 mm to (161.9, 70.8), turned to 180 degrees
- moved Q1 66.9 mm to (118.8, 86.0), turned to 180 degrees
- moved R4 63.7 mm to (113.7, 88.6), turned to 90 degrees
- moved H1 59.0 mm to (99.5, 86.5)
- moved H2 56.9 mm to (119.5, 78.0)
Connections:
- IC1 pad 3: +3V3 -> Net-(C1-Pad1)
- IC1 pad 4: IR_OUT_1 -> Net-(IC1-Pad4)
- IC2 pad 1: unconnected-(IC2-Pad1) -> VIN
- IC2 pad 2: unconnected-(IC2-Pad2) -> Net-(IC1-Pad2)
- IC2 pad 3: unconnected-(IC2-Pad3) -> Net-(C1-Pad1)
- IC2 pad 4: unconnected-(IC2-Pad4) -> Net-(IC1-Pad4)
- Q1 pad 1: Net-(Q1-Pad1) -> Net-(IC1-Pad2)
- Q1 pad 3: Net-(Q1-Pad2) -> Net-(Q1-Pad3)
- R1 pad 1: IR_IN_1 -> +3V3
- R1 pad 2: Net-(Q1-Pad2) -> Net-(C1-Pad1)
- R2 pad 1: IR_OUT_1 -> Net-(R2-Pad1)
- R2 pad 2: GND -> IR_OUT_1
- R3 pad 1: Net-(Q1-Pad1) -> Net-(C1-Pad2)
- R3 pad 2: GND -> Net-(R3-Pad2)
- R4 pad 1: VIN -> IR_IN_1
- R4 pad 2: Net-(LED1-Pad2) -> Net-(Q1-Pad2)
Routing:
- net Net-(IC1-Pad2): track 0.00 -> 90.0 mm, vias 0 -> 1
- net VIN: track 0.00 -> 70.1 mm
- net Net-(IC1-Pad4): track 0.00 -> 69.2 mm, vias 0 -> 1
- net Net-(C1-Pad1): track 0.00 -> 62.1 mm, vias 0 -> 1
- net +3V3: track 0.00 -> 54.6 mm
- net IR_OUT_1: track 0.00 -> 37.8 mm
- net IR_IN_1: track 0.00 -> 36.4 mm
- net Net-(R2-Pad1): track 0.00 -> 16.7 mm
- net Net-(Q1-Pad3): track 0.00 -> 15.0 mm
- net Net-(Q1-Pad2): track 0.00 -> 13.8 mm
- net Net-(C1-Pad2): track 0.00 -> 13.0 mm
- net Net-(R3-Pad2): track 0.00 -> 9.04 mm
- net Net-(JP1-Pad2): track 0.00 -> 6.35 mm
- net Net-(LED1-Pad2): track 0.00 -> 6.35 mm
Other:
- outline, holes or cut-outs redrawn
- board text added: "3V3"
- board text added: "Cathode"
- board text added: "Collector"
- board text added: "DRAFT"
- board text added: "Emitter"
- board text added: "IN"
- board text added: "IR LED"
- board text added: "OUT"
- board text added: "TCAR IR Board"
- board text added: "TCAR IR Board - Rev.A - (01/2022) - Scale 100%"
- board text removed: "BRAKE"
- board text removed: "EM1"
- board text removed: "EM12"
- board text removed: "EM2"
- board text removed: "EM3"
- board text removed: "EM34"
- board text removed: "EM4"
- board text removed: "M1SN"
- board text removed: "M1SPD"
- board text removed: "M2SN"
- board text removed: "M2SPD"
- board text removed: "M3SN"
- board text removed: "M3SPD"
- board text removed: "M4SN"
- board text removed: "M4SPD"
- board text removed: "STOP"
- board text removed: "TCAR MCU Board PIC24FJ - Rev.A - (01/2022) - Scale 100%"
- board text removed: "TCAR Motor Board - L298P"
