File: Kicad/ir/ir.kicad_sch (KiCad schematic)
At the start: 18 parts, among them IC1 LITEON-LTH-1550-01, IC2 LITEON-LTH-1550-01, IC3 LITEON-LTH-1550-01, Q1 BC846BS

Commit message: Update
Parts:
- removed H5, H6, H7, H8: MOUNTING-HOLE-MASK-3MM, tronixio:M3-MASK, symbol tronixio:MOUNTING-HOLE-MASK-3MM
- removed IC3: LITEON-LTH-1550-01, tronixio:zzzLTH-1550-01-HORIZONTAL, symbol tronixio:LITEON-LTH-1550-01
- removed Q1: BC846BS, tronixio:SOT-23-6, symbol tronixio:BC846BS
- removed TP1: HARWIN-S1751, tronixio:zzzHARWIN-S1751, symbol tronixio:HARWIN-S1751
- added C1, C2: C-1206, symbol tronixio:C-1206
- added JP1: HARWIN-254-M-1X02-JUMPER-VERTICAL, tronixio:HARWIN-M20-999024x, symbol tronixio:HARWIN-254-M-1X02-JUMPER-VERTICAL
- added K1: HARWIN-254-M-1X04-VERTICAL, tronixio:HARWIN-M20-999044x, symbol tronixio:HARWIN-254-M-1X04-VERTICAL
- added K2: HARWIN-254-M-1X05-VERTICAL, tronixio:HARWIN-M20-999054x, symbol tronixio:HARWIN-254-M-1X05-VERTICAL
- added K3, K4: HARWIN-254-M-1X02-VERTICAL, tronixio:HARWIN-M20-999024x, symbol tronixio:HARWIN-254-M-1X02-VERTICAL
- added Q1: (no value), symbol tronixio:ONSEMI-BC546-TO92
- added Q2: ONSEMI-BC546-TO92, tronixio:TO-92-INLINE, symbol tronixio:ONSEMI-BC546-TO92
- added R4, R5, R6, R7, R8: R-1206, symbol tronixio:R-1206
- added U1: (no value), symbol tronixio:MICROCHIP-MCP6541-DIP-08
- IC1, IC2: value LITEON-LTH-1550-01 -> (none); footprint tronixio:zzzLTH-1550-01-HORIZONTAL -> (none)
- LED1: value Power -> (none); footprint tronixio:LED-1206 -> (none); MOUSER 604-APT3216LSECKJ3RV -> (none); Mouser (none) -> 604-APT3216LSECKJ3RV
- R1: value 4K7 -> R-1206; footprint tronixio:RESISTOR-1016-TH -> (none)
- R2: value 2K7 -> R-1206; footprint tronixio:RESISTOR-1016-TH -> (none)
- R3: value 33Ω -> R-1206; footprint tronixio:RESISTOR-1016-TH -> (none)
- R9: renamed from R4; value 6K8 -> R-1206; footprint tronixio:RESISTOR-1206 -> (none)
Connections:
- net +3V3: now also R1.1, C2.1, K2.2, U1.7 (VDD); no longer IC1.3 (COLLECTOR)
- net GND: now also C2.2, K2.5, K3.1, K3.2, K4.1, K4.2, Q2.3 (E), R5.2, R6.2, R7.2, R8.2, U1.4 (GND); no longer R2.2, R3.2
- net IR_IN_1: now also K2.4, R4.1; no longer R1.1
- net IR_OUT_1: now also R2.2, K2.3, U1.6; no longer IC1.4 (EMITTER), R2.1
- net VIN: now also IC2.1 (ANODE), K1.1, K2.1
- net at IC2.2 (CATHODE): now also IC1.2 (CATHODE), K1.2, Q1.1 (C)
- net at IC2.3 (COLLECTOR): now also IC1.3 (COLLECTOR), R1.2, C1.1, K1.3
- net at IC2.4 (EMITTER): now also IC1.4 (EMITTER), JP1.1, K1.4
- net at R3.1: now also C1.2, R6.1
- new net: Q1.2 (B), Q2.1 (C), R4.2
- new net: Q1.3 (E), Q2.2 (B), R8.1
- new net: R3.2, U1.3 (+)
- new net: R2.1, R7.1, U1.2 (-)
- new net: JP1.2, R5.1
Other:
- moved on the sheet: LED1, R9

Commit message: Up
Parts:
- C1, C2: footprint (none) -> tronixio:KEMET-C322
- IC1: value (none) -> LITEON-LTH-1550-01; footprint (none) -> tronixio:zzzLTH-1550-01-HORIZONTAL
- IC2: value (none) -> LITEON-LTH-1550-01; footprint (none) -> tronixio:zzzLTH-1550-01-VERTICAL
- LED1: value (none) -> LED-1206-RED; footprint (none) -> tronixio:LED-05MM-TH
- Q1: value (none) -> ONSEMI-BC546-TO92; footprint (none) -> tronixio:TO-92-INLINE
- R1, R2, R3, R4, R5, R6, R7, R8, R9: footprint (none) -> tronixio:RESISTOR-1016-TH
- U1: value (none) -> MICROCHIP-MCP6541-DIP-08; footprint (none) -> tronixio:DIP-08-W762
Other:
- moved on the sheet: C1, IC1, IC2, JP1, K1, Q1, Q2, R1, R2, R3, R4, R5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
