File: Kicad/mcu/mcu.kicad_pcb (KiCad board)
At the start: 2 copper layers, 80 x 140 mm, 18 parts, among them IC101 LM3480-33, K301 Front, K302 Rear

Commit message: Up
Parts:
- removed G*** (x2): LOGO, tronixALL:OSHW-5MM
- added C201: 100n, tronixio:CAPACITOR-SMD-1206, F.Cu at (156.8, 97.7)
- added C202: 100n, tronixio:CAPACITOR-SMD-1206, F.Cu at (156.8, 100.7)
- added IC201: MICROCHIP-PIC24FJ64GA106-TQFP, tronixio:TQFP-64, F.Cu at (89.0, 100.0)
- added K201: ICSP, tronixio:HARWIN-M20-998034x, F.Cu at (140.3, 113.4)
- added MEMS201: MICROCHIP-DSC1001C-245760-CDFN, tronixio:CDFN-3225, F.Cu at (153.9, 114.0)
- added R201: 10K, tronixio:RESISTOR-SMD-1206, F.Cu at (156.8, 103.8)
- added R202: 1K, tronixio:RESISTOR-SMD-1206, F.Cu at (156.8, 106.8)
- added S201: Reset, tronixio:ALPS-SKRPAC, F.Cu at (148.2, 114.0)
- added X101: SYMBOL-MISC, tronixio:OSHW-5MM, F.Cu at (164.6, 99.2)
- added X102: SYMBOL-MISC, tronixio:OSHW-5MM, B.Cu at (164.6, 105.2)
- added kibuzzard-628974BE: G***, kibuzzard-628974BE, F.Cu at (100.5, 36.0)
- added kibuzzard-628974BE: G***, kibuzzard-628974BE, F.Cu at (77.6, 164.0)
- added kibuzzard-628974BE: G***, kibuzzard-628974BE, B.Cu at (100.5, 36.0)
- added kibuzzard-628974BE: G***, kibuzzard-628974BE, B.Cu at (77.6, 164.0)
- added kibuzzard-64205CDF: G***, kibuzzard-64205CDF, F.Cu at (100.5, 164.0)
- added kibuzzard-64205CDF: G***, kibuzzard-64205CDF, F.Cu at (77.6, 36.0)
- added kibuzzard-64205CDF: G***, kibuzzard-64205CDF, B.Cu at (100.5, 164.0)
- added kibuzzard-64205CDF: G***, kibuzzard-64205CDF, B.Cu at (77.6, 36.0)
- C101, C102: footprint tronixio:CAPACITOR-1206 -> tronixio:CAPACITOR-SMD-1206
- H101, H102, H103, H104, H105, H106, H107, H108: footprint tronixio:M3-MASK -> tronixio:MOUNTING-HOLE-3MM-MASK
- K301, K302: footprint tronixio:zzHARWIN-M20-782104x -> tronixio:HARWIN-M20-782104x
- LED101: value +3V3 -> Power; footprint tronixio:LED-1206 -> tronixio:LED-SMD-1206
- R101: footprint tronixio:RESISTOR-1206 -> tronixio:RESISTOR-SMD-1206
- TP101: footprint tronixio:zzzHARWIN-S1751 -> tronixio:HARWIN-S1751
- moved IC101 73.1 mm to (167.8, 116.0)
- moved R101 73.1 mm to (168.0, 112.3)
- moved C101 73.1 mm to (162.3, 112.3)
- moved LED101 73.1 mm to (162.3, 115.4)
- moved TP101 73.1 mm to (162.1, 121.8)
- moved C102 73.1 mm to (162.3, 118.5)
Connections:
- net /Encoder/BRAKE renamed /HID/BRAKE
- net /Encoder/M1_SENSE renamed /HID/M1_SENSE
- net /Encoder/M1_SPEED renamed /HID/M1_SPEED
- net /Encoder/M2_SENSE renamed /HID/M2_SENSE
- net /Encoder/M2_SPEED renamed /HID/M2_SPEED
- net /Encoder/M3_SENSE renamed /HID/M3_SENSE
- net /Encoder/M3_SPEED renamed /HID/M3_SPEED
- net /Encoder/M4_SENSE renamed /HID/M4_SENSE
- net /Encoder/M4_SPEED renamed /HID/M4_SPEED
- net /Encoder/STOP renamed /HID/STOP
- IC101 pad 1: +3V3 -> unconnected-(IC101-VO-Pad1)
- IC101 pad 2: VIN -> unconnected-(IC101-VI-Pad2)
Other:
- outline, holes or cut-outs redrawn
- board text added: "202301 - Rev.A"
- board text added: "TCAR MCU Board - L298P"
- board text added: "TCAR MCU Board PIC24FJ - Rev.A - (01/2023) - Scale 100%"
- board text removed: "202201 - Rev.A"
- board text removed: "GND"
- board text removed: "TCAR MCU Board PIC24FJ - Rev.A - (01/2022) - Scale 100%"
- board text removed: "TCAR Motor Board - L298P"
- board text removed: "VIN"
