File: Kicad/mcu/pic.kicad_sch (KiCad schematic)
At the start: 8 parts

Commit message: Up
Parts:
- C201: renamed from C?; footprint tronixio:CAPACITOR-1206 -> tronixio:CAPACITOR-SMD-1206; symbol tronixio:C-1206 -> tronixio:CAPACITOR-1206-100N-10P-X7R; Mouser (none) -> 80-C1206C104K5R; Tolerance (none) -> 10%; Voltage (none) -> 50V
- C202: renamed from C?; footprint tronixio:CAPACITOR-0805 -> tronixio:CAPACITOR-SMD-1206; symbol tronixio:C-0805 -> tronixio:CAPACITOR-1206-100N-10P-X7R; Mouser (none) -> 80-C1206C104K5R; Tolerance (none) -> 10%; Voltage (none) -> 50V
- IC201: renamed from IC?; Name PIC24FJ64GA106-TQFP -> (none)
- K201: renamed from K?; symbol tronixio:MICROCHIP-ICSP-M-2x03 -> tronixio:MICROCHIP-ICSP-M-2X03; MOUSER 855-M20-9980346 -> (none); Mouser (none) -> 855-M20-9980346
- MEMS201: renamed from MEMS?; MOUSER 998-1001CI2-024.5760 -> (none); Mouser (none) -> 998-1001CI2-024.5760; Name 24.5760MHz -> (none)
- R201: renamed from R?; footprint tronixio:RESISTOR-1206 -> tronixio:RESISTOR-SMD-1206; symbol tronixio:R-1206 -> tronixio:RESISTOR-1206-10K-5P; Mouser (none) -> 660-RK73B2BTTDD103J; Tolerance (none) -> 5%
- R202: renamed from R?; footprint tronixio:RESISTOR-1206 -> tronixio:RESISTOR-SMD-1206; symbol tronixio:R-1206 -> tronixio:RESISTOR-1206-1K-5P; Mouser (none) -> 660-RK73B2BTTDD102J; Tolerance (none) -> 5%
- S201: renamed from S?; MOUSER 688-SKRPACE010 -> (none); Mouser (none) -> 688-SKRPACE010
Connections:
- net +3V3: no longer MEMS201.4 (VDD)
- net GND: no longer K201.3 (GND), MEMS201.2 (GND)
- net MEMS: no longer MEMS201.3 (OUT)
- net PGC: no longer K201.5 (PGC)
- net PGD: no longer K201.4 (PGD)
- net ~{MCLR}: no longer K201.1 (~{MCLR})
Other:
- moved on the sheet: IC201
