File: Kicad/mcu/hid.kicad_sch (KiCad schematic)
At the start: 2 parts, among them K301 Front, K302 Rear

Commit message: Update MCU
Changed lines of the file:
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@@
     (date "01/2022")
     (rev "A")
-    (comment 1 "TCAR MCU Board - PIC24")
+    (comment 1 "TCAR MCU Board - PIC24FJ")
   )
   (wire (pts (xy 215.9 154.94) (xy 208.28 154.94))
@@
     (effects (font (size 1.27 1.27)) (justify left))
   )
+  (symbol (lib_id "tronixio:POWER-+3V3") (at 190.5 144.78 0) (unit 1)
+    (in_bom yes) (on_board yes)
+    (property "Reference" "#PWR?" (id 0) (at 190.5 157.48 0)
+      (effects (font (size 1 1)) hide)
+    )
+    (property "Value" "POWER-+3V3" (id 1) (at 190.5 154.94 0)
+      (effects (font (size 1 1)) hide)
+    )
+    (property "Footprint" "" (id 2) (at 190.5 144.78 0)
+      (effects (font (size 1 1)) hide)
+    )
+    (property "Datasheet" "" (id 3) (at 190.5 144.78 0)
+      (effects (font (size 1 1)) hide)
+    )
+    (property "Name" "+3V3" (id 4) (at 190.5 139.7 0)
+      (effects (font (size 1.15 1.15)))
+    )
+    (pin "1")
+  )
   (symbol (lib_id "tronixio:POWER-VIN") (at 254 139.7 0) (unit 1)
     (in_bom yes) (on_board yes)
@@
       (effects (font (size 1 1)) hide)
     )
+    (pin "1")
+  )
+  (symbol (lib_id "tronixio:POWER-GND") (at 190.5 162.56 0) (unit 1)
+    (in_bom yes) (on_board yes)
+    (property "Reference" "#PWR?" (id 0) (at 190.5 167.64 0)
+      (effects (font (size 1 1)) hide)
+    )
+    (property "Value" "POWER-GND" (id 1) (at 190.5 170.18 0)
+      (effects (font (size 1 1)) hide)
+    )
+    (property "Footprint" "" (id 2) (at 190.5 162.56 0)
+      (effects (font (size 1 1)) hide)
+    )
+    (property "Datasheet" "" (id 3) (at 190.5 162.56 0)
+      (effects (font (size 1 1)) hide)
+    )

Commit message: Up
Parts:
- K301, K302: footprint tronixio:zzHARWIN-M20-782104x -> tronixio:HARWIN-M20-782104x; MOUSER 855-M20-782104 -> (none); Mouser (none) -> 855-M20-782104
