File: Kicad/mcu/mcu.kicad_sch (KiCad schematic)
At the start: 14 parts, among them IC101 LM3480-33

Commit message: Update MCU
Parts:
- LED101: value +3V3 -> Power
Other:
- sheet Encoder renamed HID
- sheet MCU: file driver.kicad_sch -> pic.kicad_sch
Changed lines of the file:
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@@
     (date "01/2022")
     (rev "A")
-    (comment 1 "TCAR MCU Board - PIC24")
+    (comment 1 "TCAR MCU Board - PIC24FJ")
   )
   (junction (at 53.34 58.42) (diameter 0.9144) (color 0 0 0 0)
@@
   )
   (wire (pts (xy 172.72 180.34) (xy 172.72 190.5))
-    (stroke (width 0) (type solid) (color 0 0 0 0))
-  )
-  (wire (pts (xy 157.48 180.34) (xy 157.48 190.5))
     (stroke (width 0) (type solid) (color 0 0 0 0))
   )
@@
     (pin "1")
   )
-  (symbol (lib_id "power:PWR_FLAG") (at 157.48 190.5 180) (unit 1)
-    (in_bom yes) (on_board yes)
-    (property "Reference" "#FLG0102" (id 0) (at 157.48 188.595 0)
-      (effects (font (size 1.15 1.15)) hide)
-    )
-    (property "Value" "PWR_FLAG" (id 1) (at 157.48 186.69 0)
-      (effects (font (size 1.15 1.15)) hide)
-    )
-    (property "Footprint" "" (id 2) (at 157.48 190.5 0)
-      (effects (font (size 1 1)) hide)
-    )
-    (property "Datasheet" "~" (id 3) (at 157.48 190.5 0)
-      (effects (font (size 1 1)) hide)
-    )
-    (pin "1")
-  )
   (symbol (lib_id "tronixio:POWER-+3V3") (at 93.98 53.34 0) (unit 1)
     (in_bom yes) (on_board yes)
@@
     (pin "3")
   )
-  (symbol (lib_id "tronixio:POWER-VBAT") (at 157.48 180.34 0) (unit 1)
-    (in_bom yes) (on_board yes)
-    (property "Reference" "#PWR0108" (id 0) (at 157.48 190.5 0)
-      (effects (font (size 1 1)) hide)
-    )
-    (property "Value" "POWER-VBAT" (id 1) (at 157.48 193.04 0)
-      (effects (font (size 1 1)) hide)
-    )
-    (property "Footprint" "" (id 2) (at 157.48 180.34 0)
-      (effects (font (size 1 1)) hide)
-    )
-    (property "Datasheet" "" (id 3) (at 157.48 180.34 0)
-      (effects (font (size 1 1)) hide)
-    )
-    (property "Name" "VBAT" (id 4) (at 157.48 175.26 0)
-      (effects (font (size 1.15 1.15)))
-    )
-    (pin "1")
-  )
   (symbol (lib_id "tronixio:LED-1206-RED") (at 93.98 66.04 270) (mirror x) (unit 1)
     (in_bom yes) (on_board yes)
@@
       (effects (font (size 1.15 1.15)) (justify left))
     )
-    (property "Value" "+3V3" (id 1) (at 94.615 68.58 90)
+    (property "Value" "Power" (id 1) (at 94.615 68.58 90)
       (effects (font (size 1.15 1.15)) (justify left))
     )
@@
     (stroke (width 0.001) (type solid) (color 0 0 0 0))
     (fill (color 0 0 0 0.0000))
-    (property "Sheet name" "Encoder" (id 0) (at 93.98 146.7191 0)
+    (property "Sheet name" "HID" (id 0) (at 93.98 146.7191 0)
       (effects (font (size 1.2 1.2)) (justify left bottom))
     )
@@
       (effects (font (size 1.2 1.2)) (justify left bottom))
     )
-    (property "Sheet file" "driver.kicad_sch" (id 1) (at 43.18 182.88 0)
+    (property "Sheet file" "pic.kicad_sch" (id 1) (at 43.18 182.88 0)
       (effects (font (size 1.2 1.2)) (justify left top))
     )
@@
       (reference "#FLG0101") (unit 1) (value "PWR_FLAG") (footprint "")
     )
-    (path "/0610e5c1-7e79-4a2c-bcc8-8e76eeecda25"
-      (reference "#FLG0102") (unit 1) (value "PWR_FLAG") (footprint "")
-    )
     (path "/153c0e00-77e0-42ba-81f6-75fa564a2c4a"
       (reference "#FLG0103") (unit 1) (value "PWR_FLAG") (footprint "")
@@
       (reference "#PWR0107") (unit 1) (value "POWER-GND") (footprint "")
     )
-    (path "/d0f434dd-71f6-4972-8d50-0eb164b37036"
-      (reference "#PWR0108") (unit 1) (value "POWER-VBAT") (footprint "")
-    )
     (path "/9a3cb2cf-078a-4252-9cb7-436cdaffb870"
       (reference "#PWR0109") (unit 1) (value "POWER-VIN") (footprint "")
@@
       (reference "#PWR0304") (unit 1) (value "POWER-GND") (footprint "")
     )
+    (path "/6012b3a0-2f30-4458-8240-bd443182c6c0/0737a056-888e-4abf-8e90-747fcb02ac5b"
+      (reference "#PWR?") (unit 1) (value "POWER-GND") (footprint "")
+    )
+    (path "/56bd3a46-de12-45e9-9566-afec966f2cad/11c7caea-afa2-46e4-93dc-d94c4fd5d43e"
+      (reference "#PWR?") (unit 1) (value "POWER-+3V3") (footprint "")
+    )
+    (path "/6012b3a0-2f30-4458-8240-bd443182c6c0/20d6997e-64c7-454b-9573-baf26e1ad11b"
+      (reference "#PWR?") (unit 1) (value "POWER-+3V3") (footprint "")
+    )
+    (path "/6012b3a0-2f30-4458-8240-bd443182c6c0/3d38eca7-b037-4400-970c-46db57e3c3cb"
+      (reference "#PWR?") (unit 1) (value "POWER-+3V3") (footprint "")
+    )
+    (path "/6012b3a0-2f30-4458-8240-bd443182c6c0/3fc3a397-ec3a-4314-aa6a-44925ef4cbbe"
+      (reference "#PWR?") (unit 1) (value "POWER-GND") (footprint "")
+    )
+    (path "/6012b3a0-2f30-4458-8240-bd443182c6c0/45099ef8-b470-4f34-a90e-0a936a6b6d10"
+      (reference "#PWR?") (unit 1) (value "POWER-+3V3") (footprint "")
+    )
+    (path "/56bd3a46-de12-45e9-9566-afec966f2cad/55c0bea1-3517-4222-b109-4abebf6fdcd1"
+      (reference "#PWR?") (unit 1) (value "POWER-GND") (footprint "")
+    )
+    (path "/6012b3a0-2f30-4458-8240-bd443182c6c0/730780c7-40bd-484b-b640-ae047209b478"
+      (reference "#PWR?") (unit 1) (value "+5V") (footprint "")
+    )
+    (path "/6012b3a0-2f30-4458-8240-bd443182c6c0/ae9a2cfc-2e02-4731-9394-e388bba596f8"
+      (reference "#PWR?") (unit 1) (value "POWER-GND") (footprint "")
+    )
+    (path "/6012b3a0-2f30-4458-8240-bd443182c6c0/b4796a06-5ec1-4b7e-a305-c6447cc5c644"
+      (reference "#PWR?") (unit 1) (value "GND") (footprint "")
+    )
+    (path "/6012b3a0-2f30-4458-8240-bd443182c6c0/e525b640-a490-46b0-aa2a-5838f1d12b7d"
+      (reference "#PWR?") (unit 1) (value "POWER-GND") (footprint "")
+    )
+    (path "/6012b3a0-2f30-4458-8240-bd443182c6c0/fedb7d4b-8ca2-493c-b9a1-22e781d6d436"
+      (reference "#PWR?") (unit 1) (value "GND") (footprint "")
+    )
     (path "/3e9b3e5f-7172-4412-9e9a-af7341007fe7"
       (reference "C101") (unit 1) (value "1µ") (footprint "tronixio:CAPACITOR-1206")
@@
       (reference "C102") (unit 1) (value "1µ") (footprint "tronixio:CAPACITOR-1206")
     )
+    (path "/6012b3a0-2f30-4458-8240-bd443182c6c0/85c4eb9a-1efe-40fd-86af-36f89108b5f9"
+      (reference "C?") (unit 1) (value "100n") (footprint "tronixio:CAPACITOR-0805")
+    )
+    (path "/6012b3a0-2f30-4458-8240-bd443182c6c0/d9c1c6f8-c198-49f9-bff0-eab2393a0053"
+      (reference "C?") (unit 1) (value "100n") (footprint "tronixio:CAPACITOR-1206")
+    )
     (path "/bd7dbed2-53d4-417c-9458-85252bdbb186"
       (reference "H101") (unit 1) (value "MOUNTING-HOLE-MASK-3MM") (footprint "tronixio:M3-MASK")
@@
       (reference "IC101") (unit 1) (value "LM3480-33") (footprint "tronixio:SOT-23-3")
     )
+    (path "/6012b3a0-2f30-4458-8240-bd443182c6c0/a2a055dc-7e5e-409c-bc15-cb64711b5b65"
+      (reference "IC?") (unit 1) (value "MICROCHIP-PIC24FJ64GA106-TQFP") (footprint "tronixio:TQFP-64")
+    )
     (path "/56bd3a46-de12-45e9-9566-afec966f2cad/9f0e67b6-f260-4089-b2ad-142f7a74e82f"
       (reference "K301") (unit 1) (value "Front") (footprint "tronixio:zzHARWIN-M20-782104x")
@@
       (reference "K302") (unit 1) (value "Rear") (footprint "tronixio:zzHARWIN-M20-782104x")
     )
+    (path "/6012b3a0-2f30-4458-8240-bd443182c6c0/fd27925d-9b2e-4663-bdb7-e46b9715b801"
+      (reference "K?") (unit 1) (value "ICSP") (footprint "tronixio:HARWIN-M20-998034x")
+    )
     (path "/d60193f4-8481-4abd-b144-cbba3dc6e1a6"
-      (reference "LED101") (unit 1) (value "+3V3") (footprint "tronixio:LED-1206")
+      (reference "LED101") (unit 1) (value "Power") (footprint "tronixio:LED-1206")
+    )
+    (path "/6012b3a0-2f30-4458-8240-bd443182c6c0/d789eb5c-7750-4e88-bd51-088f1d8d4899"
+      (reference "MEMS?") (unit 1) (value "MICROCHIP-DSC1001C-245760-CDFN") (footprint "tronixio:CDFN-3225")
     )
     (path "/8003b8b6-1f3c-47e9-a876-bee51c25ef20"
       (reference "R101") (unit 1) (value "6K8") (footprint "tronixio:RESISTOR-1206")
     )
+    (path "/6012b3a0-2f30-4458-8240-bd443182c6c0/6bdf4c09-0d97-4f84-a45b-4830c8cb3132"
+      (reference "R?") (unit 1) (value "10K") (footprint "tronixio:RESISTOR-1206")
+    )
+    (path "/6012b3a0-2f30-4458-8240-bd443182c6c0/d0b8883f-56d3-436a-a178-a658388f963b"
+      (reference "R?") (unit 1) (value "1K") (footprint "tronixio:RESISTOR-1206")
+    )
+    (path "/6012b3a0-2f30-4458-8240-bd443182c6c0/2a6f1b1e-6809-43d7-b0c5-e4424e33d333"
+      (reference "S?") (unit 1) (value "Reset") (footprint "tronixio:ALPS-SKRPAC")
+    )
     (path "/6ab23ab0-73e6-4657-ab97-4027cb5eba59"

Commit message: Up
Parts:
- added X101, X102: SYMBOL-MISC, tronixio:OSHW-5MM, symbol tronixio:OSHW-5MM
- C101, C102: footprint tronixio:CAPACITOR-1206 -> tronixio:CAPACITOR-SMD-1206; symbol tronixio:C-1206 -> tronixio:CAPACITOR-1206-1U-10P-X7R; Mouser (none) -> 80-C1206C105K5R; Tolerance (none) -> 10%; Voltage (none) -> 50V
- H101, H102, H103, H104, H105, H106, H107, H108: footprint tronixio:M3-MASK -> tronixio:MOUNTING-HOLE-3MM-MASK; symbol tronixio:MOUNTING-HOLE-MASK-3MM -> tronixio:MOUNTING-HOLE-3MM-MASK
- IC101: symbol tronixio:LM3480-33-SOT -> tronixio:TI-LM3480-33-SOT-23; MOUSER 926-LM3480IM33.3NOPB -> (none); Mouser (none) -> 926-LM3480IM33.3NOPB
- LED101: footprint tronixio:LED-1206 -> tronixio:LED-SMD-1206; symbol tronixio:LED-1206-RED -> tronixio:KINGBRIGHT-LED-1206-RED; MOUSER 604-APT3216LSECKJ3RV -> (none); Mouser (none) -> 604-APT3216LSECKJ3RV
- R101: footprint tronixio:RESISTOR-1206 -> tronixio:RESISTOR-SMD-1206; symbol tronixio:R-1206 -> tronixio:RESISTOR-1206-6K8-5P; Mouser (none) -> 660-RK73B2BTTDD682J; Tolerance (none) -> 5%
- TP101: footprint tronixio:zzzHARWIN-S1751 -> tronixio:HARWIN-S1751; MOUSER 855-S1751-46 -> (none); Mouser (none) -> 855-S1751-46
Connections:
- net +3V3: no longer IC101.1 (VO)
- net VIN: no longer IC101.2 (VI)
Other:
- title: Power -> Root & Power

Commit message: Up
Parts:
- removed C101, C102: 1µ, tronixio:CAPACITOR-SMD-1206, symbol tronixio:CAPACITOR-1206-1U-10P-X7R
- removed H101, H102, H103, H104, H105, H106, H107, H108: MOUNTING-HOLE-MASK-3MM, tronixio:MOUNTING-HOLE-3MM-MASK, symbol tronixio:MOUNTING-HOLE-3MM-MASK
- removed IC101: LM3480-33, tronixio:SOT-23-3, symbol tronixio:TI-LM3480-33-SOT-23
- removed LED101: Power, tronixio:LED-SMD-1206, symbol tronixio:KINGBRIGHT-LED-1206-RED
- removed R101: 6K8, tronixio:RESISTOR-SMD-1206, symbol tronixio:RESISTOR-1206-6K8-5P
- removed TP101: HARWIN-S1751, tronixio:HARWIN-S1751, symbol tronixio:HARWIN-S1751
- removed X101, X102: SYMBOL-MISC, tronixio:OSHW-5MM, symbol tronixio:OSHW-5MM
- added C201, C202: 100n, tronixio:CAPACITOR-SMD-1206, symbol tronixio:CAPACITOR-1206-100N-10P-X7R
- added IC201: MICROCHIP-PIC24FJ64GA106-TQFP, tronixio:TQFP-64, symbol tronixio:MICROCHIP-PIC24FJ64GA106-TQFP
- added K201: ICSP, tronixio:HARWIN-M20-998034x, symbol tronixio:MICROCHIP-ICSP-M-2X03
- added MEMS201: MICROCHIP-DSC1001C-245760-CDFN, tronixio:CDFN-3225, symbol tronixio:MICROCHIP-DSC1001C-245760-CDFN
- added R201: 10K, tronixio:RESISTOR-SMD-1206, symbol tronixio:RESISTOR-1206-10K-5P
- added R202: 1K, tronixio:RESISTOR-SMD-1206, symbol tronixio:RESISTOR-1206-1K-5P
- added S201: Reset, tronixio:ALPS-SKRPAC, symbol tronixio:ALPS-SKRPAC
Connections:
- net +3V3: now also C202.1, K201.2 (VDD)
- net GND: now also C201.2, C202.2, S201.1, S201.2
- new net: C201.1, R201.1, R202.2, S201.3, S201.4
- new net +5V: R201.2
- new net ~{MCLR}: R202.1
- no-connect marks 0 -> 1
Other:
- removed sheet HID
- removed sheet MCU
- note added: "Dans la mesure du possible utiliser les pins non 5v pour la motor board, reserver les 5v capabilities pour les capteurs externes"
- title: Root & Power -> MCU - PIC24FJxxxGA106
